Commit message: gripper added

File: Assets/kuka_kr3_support/urdf/kr3r540.urdf (robot description, URDF)
Before this commit: robot kuka_kr3r540, 10 links, 9 joints
Links:
- added link gripper_base_link, mass 0.25; collision mesh filename=package://wsg_50_simulation/meshes/WSG50_110.stl scale=1 1 1; visual mesh filename=package://wsg_50_simulation/meshes/WSG50_110.stl scale=1 1 1
- added link gripper_center
- added link gripper_finger_left, mass 0.1; collision mesh filename=package://wsg_50_simulation/meshes/WSG-FMF.stl scale=0.001 0.001 0.001; visual mesh filename=package://wsg_50_simulation/meshes/WSG-FMF.stl scale=0.001 0.001 0.001
- added link gripper_finger_right, mass 0.1; collision mesh filename=package://wsg_50_simulation/meshes/WSG-FMF.stl scale=0.001 0.001 0.001; visual mesh filename=package://wsg_50_simulation/meshes/WSG-FMF.stl scale=0.001 0.001 0.001
- added link gripper_gripper_left, mass 0.1; collision mesh filename=package://wsg_50_simulation/meshes/GUIDE_WSG50_110.stl scale=0.001 0.001 0.001; visual mesh filename=package://wsg_50_simulation/meshes/GUIDE_WSG50_110.stl scale=0.001 0.001 0.001
- added link gripper_gripper_right, mass 0.1; collision mesh filename=package://wsg_50_simulation/meshes/GUIDE_WSG50_110.stl scale=0.001 0.001 0.001; visual mesh filename=package://wsg_50_simulation/meshes/GUIDE_WSG50_110.stl scale=0.001 0.001 0.001
Joints:
- added joint gripper_anterior_gripper_joint: type fixed, parent tool0, child gripper_base_link, origin xyz=0 0 0 rpy=0 0 0
- added joint gripper_center_joint: type fixed, parent gripper_base_link, child gripper_center, origin xyz=0 0 -0.017 rpy=0 0 0
- added joint gripper_finger_left_joint: type prismatic, parent gripper_base_link, child gripper_gripper_left, origin xyz=0 0 0 rpy=0 0 0, axis 1 0 0, limit lower=-0.055 upper=-0.0027 effort=1.0 velocity=1.0
- added joint gripper_finger_right_joint: type prismatic, parent gripper_base_link, child gripper_gripper_right, origin xyz=0 0 0 rpy=0 0 3.14159, axis -1 0 0, limit lower=0.0027 upper=0.055 effort=1.0 velocity=1.0
- added joint gripper_guide_joint_finger_left: type fixed, parent gripper_gripper_left, child gripper_finger_left, origin xyz=0 0 -0.017 rpy=0 0 0, axis 1 0 0, limit effort=100 velocity=100
- added joint gripper_guide_joint_finger_right: type fixed, parent gripper_gripper_right, child gripper_finger_right, origin xyz=0 0 -0.017 rpy=0 0 0, axis 1 0 0, limit effort=100 velocity=100
