Commit message: minor changes

File: Assets/kr3r540/test/kr3r540_v2.urdf (robot description, URDF)
Before this commit: robot kuka_kr3r540, 16 links, 15 joints
Links:
- link link_6: mass 3 -> None
Joints:
- joint joint_a1: limit lower=-2.9670597283903604 upper=2.9670597283903604 effort=1.0 velocity=9.250245035569947 -> lower=-2.9670597283903604 upper=2.9670597283903604 effort=0 velocity=9.250245035569947
- joint joint_a2: limit lower=-2.9670597283903604 upper=0.8726646259971648 effort=1.0 velocity=9.232791743050003 -> lower=-2.9670597283903604 upper=0.8726646259971648 effort=1000 velocity=9.232791743050003
- joint joint_a3: limit lower=-1.9198621771937625 upper=2.705260340591211 effort=100 velocity=9.389871375729493 -> lower=-1.9198621771937625 upper=2.705260340591211 effort=0 velocity=9.389871375729493
- joint joint_a4: limit lower=-3.0543261909900767 upper=3.0543261909900767 effort=100 velocity=10.471975511965978 -> lower=-3.0543261909900767 upper=3.0543261909900767 effort=0 velocity=10.471975511965978
- joint joint_a5: limit lower=-2.0943951023931953 upper=2.0943951023931953 effort=100 velocity=10.471975511965978 -> lower=-2.0943951023931953 upper=2.0943951023931953 effort=0 velocity=10.471975511965978
- joint joint_a6: limit lower=-6.1086523819801535 upper=6.1086523819801535 effort=100 velocity=13.962634015954636 -> lower=-6.1086523819801535 upper=6.1086523819801535 effort=0 velocity=13.962634015954636
