Commit message: Kr3 v3 added, corrected max force, stifness and dampening
kr3 urdf v3 created

File: Assets/kr3r540/kr3r540_v2.urdf (robot description, URDF)
Before this commit: robot kuka_kr3r540, 16 links, 15 joints
Joints:
- joint joint_a1: limit lower=-2.9670597283903604 upper=2.9670597283903604 effort=1.0 velocity=9.250245035569947 -> lower=-2.9670597283903604 upper=2.9670597283903604 effort=100 velocity=9.250245035569947
- joint joint_a2: limit lower=-2.9670597283903604 upper=0.8726646259971648 effort=1.0 velocity=9.232791743050003 -> lower=-2.9670597283903604 upper=0.8726646259971648 effort=100 velocity=9.232791743050003
