Commit message: limit effort set to 100

File: Assets/kr4r600/kr4r600_v1.urdf (robot description, URDF)
Before this commit: robot kuka_kr4r600, 9 links, 8 joints
Joints:
- joint joint_a1: limit lower=-2.9670597283903604 upper=2.9670597283903604 effort=0 velocity=9.250245035569947 -> lower=-2.9670597283903604 upper=2.9670597283903604 effort=100 velocity=9.250245035569947
- joint joint_a2: limit lower=-3.4033920413889427 upper=0.6981317007977318 effort=0 velocity=9.232791743050003 -> lower=-3.4033920413889427 upper=0.6981317007977318 effort=100 velocity=9.232791743050003
- joint joint_a3: limit lower=-2.007128639793479 upper=2.6179938779914944 effort=0 velocity=9.389871375729493 -> lower=-2.007128639793479 upper=2.6179938779914944 effort=100 velocity=9.389871375729493
- joint joint_a4: limit lower=-3.2288591161895095 upper=3.2288591161895095 effort=0 velocity=10.471975511965978 -> lower=-3.2288591161895095 upper=3.2288591161895095 effort=100 velocity=10.471975511965978
- joint joint_a5: limit lower=-2.0943951023931953 upper=2.0943951023931953 effort=0 velocity=10.471975511965978 -> lower=-2.0943951023931953 upper=2.0943951023931953 effort=100 velocity=10.471975511965978
- joint joint_a6: limit lower=-6.1086523819801535 upper=6.1086523819801535 effort=0 velocity=13.962634015954636 -> lower=-6.1086523819801535 upper=6.1086523819801535 effort=100 velocity=13.962634015954636
