Commit message: urdf for tools + base config

File: src/kr3_config_dispenser/config/gazebo_kuka_kr3r540.urdf (robot description, URDF)
Before this commit: robot kuka_kr3r540, 11 links, 10 joints
Links:
- link base_link_gripper: geometry collision mesh filename=package://kuka_kr3_support/meshes/kr3r540/collision/Dispens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 scale=0.001 0.001 0.001; visual mesh filename=package://kuka_kr3_support/meshes/kr3r540/visual/Dispenser.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 scale=0.001 0.001 0.001

File: src/kuka_kr3_support/urdf/kr3r540_dispenser.urdf (robot description, URDF)
Before this commit: robot kuka_kr3r540, 11 links, 10 joints
Links:
- link base_link_gripper: geometry collision mesh filename=package://kuka_kr3_support/meshes/kr3r540/collision/Dispens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 scale=0.001 0.001 0.001; visual mesh filename=package://kuka_kr3_support/meshes/kr3r540/visual/Dispenser.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 scale=0.001 0.001 0.001

File: src/kuka_kr3_support/urdf/kr3r540_pipette.urdf (robot description, URDF)
Before this commit: robot kuka_kr3r540, 11 links, 10 joints
Links:
- link base_link_gripper: geometry collision mesh filename=package://kuka_kr3_support/meshes/kr3r540/collision/Pipette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 scale=0.001 0.001 0.001; visual mesh filename=package://kuka_kr3_support/meshes/kr3r540/visual/Pipette.stl scale=0.001 0.001 0.001
