Commit message: Assets added

File: src/schunk_25nnb/urdf/schunk_25nnb.urdf (robot description, URDF)
Before this commit: robot schunk_25nnb, 3 links, 2 joints
Links:
- link base_link: mass 3.08428949350963E-05 -> 3.0843E-05
- link left_link: mass 9.1881E-07 -> 0.016862
- link right_link: mass 9.1881E-07 -> 0.016862
