Commit message: Added pipette and dispenser to xacro macro and xacro tools

File: src/kuka_kr3_support/urdf/kr3r540_macro_v2.xacro (robot description, xacro)
@@ -16,4 +16,9 @@
           <mesh filename="package://kuka_kr3_support/meshes/kr3r540/collision/base_link.stl" />
         </geometry>
+        <inertial>
+          <origin rpy="0 0 0" xyz="0 0 0"/>
+          <mass value="8.45"/>
+          <inertia ixx="0.09" ixy="0.0" ixz="-0.02" iyy="0.11" iyz="0.0" izz="0.05"/>
+        </inertial>
       </collision>
     </link>
@@ -31,4 +36,9 @@
           <mesh filename="package://kuka_kr3_support/meshes/kr3r540/collision/link_1.stl" />
         </geometry>
+        <inertial>
+          <origin rpy="0 0 0" xyz="0 0 0"/>
+          <mass value="4.46"/>
+          <inertia ixx="0.24" ixy="0.0" ixz="0.0" iyy="0.24" iyz="0.0" izz="0.02"/>
+        </inertial>
       </collision>
     </link>
@@ -45,4 +55,9 @@
           <mesh filename="package://kuka_kr3_support/meshes/kr3r540/collision/link_2.stl" />
         </geometry>
+        <inertial>
+          <origin rpy="0 0 0" xyz="0 0 0"/>
+          <mass value="9.11"/>
+          <inertia ixx="0.065" ixy="0.0" ixz="0.0" iyy="0.065" iyz="0.0" izz="0.02"/>
+        </inertial>
       </collision>
     </link>
@@ -60,4 +75,9 @@
           <mesh filename="package://kuka_kr3_support/meshes/kr3r540/collision/link_3.stl" />
         </geometry>
+        <inertial>
+          <origin rpy="0 0 0" xyz="0 0 0"/>
+          <mass value="2.2"/>
+          <inertia ixx="0.64" ixy="0.0" ixz="0.05" iyy="0.64" iyz="0.0" izz="0.01"/>
+        </inertial>
       </collision>
     </link>
@@ -75,4 +95,9 @@
           <mesh filename="package://kuka_kr3_support/meshes/kr3r540/collision/link_4.stl" />
         </geometry>
+        <inertial>
+          <origin rpy="0 0 0" xyz="0 0 0"/>
+          <mass value="1.5"/>
+          <inertia ixx="0.45" ixy="0.0" ixz="0.15" iyy="0.5" iyz="0.0" izz="0.05"/>
+        </inertial>
       </collision>
     </link>
@@ -90,4 +115,9 @@
           <mesh filename="package://kuka_kr3_support/meshes/kr3r540/collision/link_5.stl" />
         </geometry>
+        <inertial>
+          <origin rpy="0 0 0" xyz="0 0 0"/>
+          <mass value="0.75"/>
+          <inertia ixx="0.23" ixy="0.0" ixz="0.1" iyy="0.28" iyz="0.0" izz="0.05"/>
+        </inertial>
       </collision>
     </link>
@@ -105,4 +135,9 @@
           <mesh filename="package://kuka_kr3_support/meshes/kr3r540/collision/link_6.stl" />
         </geometry>
+        <inertial>
+          <origin rpy="0 0 0" xyz="0 0 0"/>
+          <mass value="0.026"/>
+          <inertia ixx="0.01" ixy="0.0" ixz="0.0" iyy="0.01" iyz="0" izz="0"/>
+        </inertial>
       </collision>
     </link>
@@ -114,12 +149,12 @@
       <child link="${prefix}link_1"/>
       <axis xyz="0 0 -1"/>
-      <limit lower="${radians(-170)}" upper="${radians(170)}" effort="0" velocity="${radians(530)}"/>
+      <limit lower="${radians(-170)}" upper="${radians(170)}" effort="100" velocity="${radians(530)}"/>
     </joint>
     <joint name="${prefix}joint_a2" type="revolute">
-      <origin xyz="0.020 0 0" rpy="0 0 0"/>
+      <origin xyz="0.020 0 0" rpy="0 -1 0"/>
       <parent link="${prefix}link_1"/>
       <child link="${prefix}link_2"/>
       <axis xyz="0 1 0"/>
-      <limit lower="${radians(-170)}" upper="${radians(50)}" effort="0" velocity="${radians(529)}"/>
+      <limit lower="${radians(-170)}" upper="${radians(50)}" effort="100" velocity="${radians(529)}"/>
     </joint>
     <joint name="${prefix}joint_a3" type="revolute">
@@ -128,5 +163,5 @@
       <child link="${prefix}link_3"/>
       <axis xyz="0 1 0"/>
-      <limit lower="${radians(-110)}" upper="${radians(155)}" effort="0" velocity="${radians(538)}"/>
+      <limit lower="${radians(-110)}" upper="${radians(155)}" effort="100" velocity="${radians(538)}"/>
     </joint>
     <joint name="${prefix}joint_a4" type="revolute">
@@ -135,5 +170,5 @@
       <child link="${prefix}link_4"/>
       <axis xyz="-1 0 0"/>
-      <limit lower="${radians(-175)}" upper="${radians(175)}" effort="0" velocity="${radians(600)}"/>
+      <limit lower="${radians(-175)}" upper="${radians(175)}" effort="100" velocity="${radians(600)}"/>
     </joint>
     <joint name="${prefix}joint_a5" type="revolute">
@@ -142,5 +177,5 @@
       <child link="${prefix}link_5"/>
       <axis xyz="0 1 0"/>
-      <limit lower="${radians(-120)}" upper="${radians(120)}" effort="0" velocity="${radians(600)}"/>
+      <limit lower="${radians(-120)}" upper="${radians(120)}" effort="100" velocity="${radians(600)}"/>
     </joint>
     <joint name="${prefix}joint_a6" type="revolute">
@@ -149,5 +184,5 @@
       <child link="${prefix}link_6"/>
       <axis xyz="-1 0 0"/>
-      <limit lower="${radians(-350)}" upper="${radians(350)}" effort="0" velocity="${radians(800)}"/>
+      <limit lower="${radians(-350)}" upper="${radians(350)}" effort="100" velocity="${radians(800)}"/>
     </joint>
     <joint name="${prefix}joint_a6-tool0" type="fixed">
