Commit message: Added pipette and dispenser to xacro macro and xacro tools

File: src/kuka_multiple_arms/robot_description/kuka_multiple_arms.urdf (robot description, URDF)
Before this commit: robot kuka_multiple_arms, 55 links, 54 joints
Links:
- removed link kr3_disp_base_link
- removed link kr3_disp_flange
- removed link kr3_disp_link_1
- removed link kr3_disp_link_2
- removed link kr3_disp_link_3
- removed link kr3_disp_link_4
- removed link kr3_disp_link_5
- removed link kr3_disp_link_6
- removed link kr3_disp_tool0
- removed link kr3_pip_base_link
- removed link kr3_pip_flange
- removed link kr3_pip_link_1
- removed link kr3_pip_link_2
- removed link kr3_pip_link_3
- removed link kr3_pip_link_4
- removed link kr3_pip_link_5
- removed link kr3_pip_link_6
- removed link kr3_pip_tool0
- removed link kr3_pp1_base_link
- removed link kr3_pp1_flange
- removed link kr3_pp1_link_1
- removed link kr3_pp1_link_2
- removed link kr3_pp1_link_3
- removed link kr3_pp1_link_4
- removed link kr3_pp1_link_5
- removed link kr3_pp1_link_6
- removed link kr3_pp1_schunk_base_link
- removed link kr3_pp1_schunk_left_link
- removed link kr3_pp1_schunk_right_link
- removed link kr3_pp1_tool0
- removed link kr3_pp2_base_link
- removed link kr3_pp2_flange
- removed link kr3_pp2_link_1
- removed link kr3_pp2_link_2
- removed link kr3_pp2_link_3
- removed link kr3_pp2_link_4
- removed link kr3_pp2_link_5
- removed link kr3_pp2_link_6
- removed link kr3_pp2_schunk_base_link
- removed link kr3_pp2_schunk_left_link
- removed link kr3_pp2_schunk_right_link
- removed link kr3_pp2_tool0
- removed link kr4_pp3_base_link
- removed link kr4_pp3_kr4_pp3_base_link
- removed link kr4_pp3_kr4_pp3_left_link
- removed link kr4_pp3_kr4_pp3_right_link
- removed link kr4_pp3_link_1
- removed link kr4_pp3_link_2
- removed link kr4_pp3_link_3
- removed link kr4_pp3_link_4
- removed link kr4_pp3_link_5
- removed link kr4_pp3_link_6
- removed link kr4_pp3_tool0
- added link kr3_1_base_link; collision mesh filename=package://kuka_kr3_support/meshes/kr3r540/collision/base_li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; visual mesh filename=package://kuka_kr3_support/meshes/kr3r540/visual/base_link.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
- added link kr3_1_flange
- added link kr3_1_link_1; collision mesh filename=package://kuka_kr3_support/meshes/kr3r540/collision/link_1.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; visual mesh filename=package://kuka_kr3_support/meshes/kr3r540/visual/link_1.stl
- added link kr3_1_link_2; collision mesh filename=package://kuka_kr3_support/meshes/kr3r540/collision/link_2.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; visual mesh filename=package://kuka_kr3_support/meshes/kr3r540/visual/link_2.stl
- added link kr3_1_link_3; collision mesh filename=package://kuka_kr3_support/meshes/kr3r540/collision/link_3.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; visual mesh filename=package://kuka_kr3_support/meshes/kr3r540/visual/link_3.stl
- added link kr3_1_link_4; collision mesh filename=package://kuka_kr3_support/meshes/kr3r540/collision/link_4.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; visual mesh filename=package://kuka_kr3_support/meshes/kr3r540/visual/link_4.stl
- added link kr3_1_link_5; collision mesh filename=package://kuka_kr3_support/meshes/kr3r540/collision/link_5.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; visual mesh filename=package://kuka_kr3_support/meshes/kr3r540/visual/link_5.stl
- added link kr3_1_link_6; collision mesh filename=package://kuka_kr3_support/meshes/kr3r540/collision/link_6.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; visual mesh filename=package://kuka_kr3_support/meshes/kr3r540/visual/link_6.stl
- added link kr3_1_schunk_base_link, mass 3.08428949350963E-05; collision mesh filename=package://schunk_25nnb/meshes/base_link.STL; visual mesh filename=package://schunk_25nnb/meshes/base_link.STL
- added link kr3_1_schunk_left_link, mass 9.1881E-07; collision mesh filename=package://schunk_25nnb/meshes/left_link.STL; visual mesh filename=package://schunk_25nnb/meshes/left_link.STL
- added link kr3_1_schunk_right_link, mass 9.1881E-07; collision mesh filename=package://schunk_25nnb/meshes/right_link.STL; visual mesh filename=package://schunk_25nnb/meshes/right_link.STL
- added link kr3_1_tool0
- added link kr3_2_base_link; collision mesh filename=package://kuka_kr3_support/meshes/kr3r540/collision/base_li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; visual mesh filename=package://kuka_kr3_support/meshes/kr3r540/visual/base_link.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
- added link kr3_2_flange
- added link kr3_2_link_1; collision mesh filename=package://kuka_kr3_support/meshes/kr3r540/collision/link_1.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; visual mesh filename=package://kuka_kr3_support/meshes/kr3r540/visual/link_1.stl
- added link kr3_2_link_2; collision mesh filename=package://kuka_kr3_support/meshes/kr3r540/collision/link_2.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; visual mesh filename=package://kuka_kr3_support/meshes/kr3r540/visual/link_2.stl
- added link kr3_2_link_3; collision mesh filename=package://kuka_kr3_support/meshes/kr3r540/collision/link_3.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; visual mesh filename=package://kuka_kr3_support/meshes/kr3r540/visual/link_3.stl
- added link kr3_2_link_4; collision mesh filename=package://kuka_kr3_support/meshes/kr3r540/collision/link_4.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; visual mesh filename=package://kuka_kr3_support/meshes/kr3r540/visual/link_4.stl
- added link kr3_2_link_5; collision mesh filename=package://kuka_kr3_support/meshes/kr3r540/collision/link_5.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; visual mesh filename=package://kuka_kr3_support/meshes/kr3r540/visual/link_5.stl
- added link kr3_2_link_6; collision mesh filename=package://kuka_kr3_support/meshes/kr3r540/collision/link_6.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; visual mesh filename=package://kuka_kr3_support/meshes/kr3r540/visual/link_6.stl
- added link kr3_2_schunk_base_link, mass 3.08428949350963E-05; collision mesh filename=package://schunk_25nnb/meshes/base_link.STL; visual mesh filename=package://schunk_25nnb/meshes/base_link.STL
- added link kr3_2_schunk_left_link, mass 9.1881E-07; collision mesh filename=package://schunk_25nnb/meshes/left_link.STL; visual mesh filename=package://schunk_25nnb/meshes/left_link.STL
- added link kr3_2_schunk_right_link, mass 9.1881E-07; collision mesh filename=package://schunk_25nnb/meshes/right_link.STL; visual mesh filename=package://schunk_25nnb/meshes/right_link.STL
- added link kr3_2_tool0
- added link kr3_3_base_link; collision mesh filename=package://kuka_kr3_support/meshes/kr3r540/collision/base_li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; visual mesh filename=package://kuka_kr3_support/meshes/kr3r540/visual/base_link.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
- added link kr3_3_flange
- added link kr3_3_link_1; collision mesh filename=package://kuka_kr3_support/meshes/kr3r540/collision/link_1.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; visual mesh filename=package://kuka_kr3_support/meshes/kr3r540/visual/link_1.stl
- added link kr3_3_link_2; collision mesh filename=package://kuka_kr3_support/meshes/kr3r540/collision/link_2.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; visual mesh filename=package://kuka_kr3_support/meshes/kr3r540/visual/link_2.stl
- added link kr3_3_link_3; collision mesh filename=package://kuka_kr3_support/meshes/kr3r540/collision/link_3.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; visual mesh filename=package://kuka_kr3_support/meshes/kr3r540/visual/link_3.stl
- added link kr3_3_link_4; collision mesh filename=package://kuka_kr3_support/meshes/kr3r540/collision/link_4.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; visual mesh filename=package://kuka_kr3_support/meshes/kr3r540/visual/link_4.stl
- added link kr3_3_link_5; collision mesh filename=package://kuka_kr3_support/meshes/kr3r540/collision/link_5.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; visual mesh filename=package://kuka_kr3_support/meshes/kr3r540/visual/link_5.stl
- added link kr3_3_link_6; collision mesh filename=package://kuka_kr3_support/meshes/kr3r540/collision/link_6.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; visual mesh filename=package://kuka_kr3_support/meshes/kr3r540/visual/link_6.stl
- added link kr3_3_pip_base_link, mass 3.08428949350963E-05; collision mesh filename=package://kuka_kr3_support/meshes/kr3r540/collision/Pipette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 scale=0.001 0.001 0.001; visual mesh filename=package://kuka_kr3_support/meshes/kr3r540/visual/Pipette.stl scale=0.001 0.001 0.001
- added link kr3_3_tool0
- added link kr3_4_base_link; collision mesh filename=package://kuka_kr3_support/meshes/kr3r540/collision/base_li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; visual mesh filename=package://kuka_kr3_support/meshes/kr3r540/visual/base_link.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
- added link kr3_4_disp_base_link, mass 3.08428949350963E-05; collision mesh filename=package://kuka_kr3_support/meshes/kr3r540/collision/Dispens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 scale=0.001 0.001 0.001; visual mesh filename=package://kuka_kr3_support/meshes/kr3r540/visual/Dispenser.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 scale=0.001 0.001 0.001
- added link kr3_4_flange
- added link kr3_4_link_1; collision mesh filename=package://kuka_kr3_support/meshes/kr3r540/collision/link_1.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; visual mesh filename=package://kuka_kr3_support/meshes/kr3r540/visual/link_1.stl
- added link kr3_4_link_2; collision mesh filename=package://kuka_kr3_support/meshes/kr3r540/collision/link_2.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; visual mesh filename=package://kuka_kr3_support/meshes/kr3r540/visual/link_2.stl
- added link kr3_4_link_3; collision mesh filename=package://kuka_kr3_support/meshes/kr3r540/collision/link_3.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; visual mesh filename=package://kuka_kr3_support/meshes/kr3r540/visual/link_3.stl
- added link kr3_4_link_4; collision mesh filename=package://kuka_kr3_support/meshes/kr3r540/collision/link_4.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; visual mesh filename=package://kuka_kr3_support/meshes/kr3r540/visual/link_4.stl
- added link kr3_4_link_5; collision mesh filename=package://kuka_kr3_support/meshes/kr3r540/collision/link_5.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; visual mesh filename=package://kuka_kr3_support/meshes/kr3r540/visual/link_5.stl
- added link kr3_4_link_6; collision mesh filename=package://kuka_kr3_support/meshes/kr3r540/collision/link_6.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; visual mesh filename=package://kuka_kr3_support/meshes/kr3r540/visual/link_6.stl
- added link kr3_4_tool0
- added link kr4_5_base_link; collision mesh filename=package://kuka_kr4_support/meshes/kr4r600/collision/base_li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; visual mesh filename=package://kuka_kr4_support/meshes/kr4r600/visual/base_link.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
- added link kr4_5_link_1; collision mesh filename=package://kuka_kr4_support/meshes/kr4r600/collision/link_1.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; visual mesh filename=package://kuka_kr4_support/meshes/kr4r600/visual/link_1.stl
- added link kr4_5_link_2; collision mesh filename=package://kuka_kr4_support/meshes/kr4r600/collision/link_2.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; visual mesh filename=package://kuka_kr4_support/meshes/kr4r600/visual/link_2.stl
- added link kr4_5_link_3; collision mesh filename=package://kuka_kr4_support/meshes/kr4r600/collision/link_3.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; visual mesh filename=package://kuka_kr4_support/meshes/kr4r600/visual/link_3.stl
- added link kr4_5_link_4; collision mesh filename=package://kuka_kr4_support/meshes/kr4r600/collision/link_4.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; visual mesh filename=package://kuka_kr4_support/meshes/kr4r600/visual/link_4.stl
- added link kr4_5_link_5; collision mesh filename=package://kuka_kr4_support/meshes/kr4r600/collision/link_5.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; visual mesh filename=package://kuka_kr4_support/meshes/kr4r600/visual/link_5.stl
- added link kr4_5_link_6; collision mesh filename=package://kuka_kr4_support/meshes/kr4r600/collision/link_6.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; visual mesh filename=package://kuka_kr4_support/meshes/kr4r600/visual/link_6.stl
- added link kr4_5_schunk_base_link, mass 3.08428949350963E-05; collision mesh filename=package://schunk_25nnb/meshes/base_link.STL; visual mesh filename=package://schunk_25nnb/meshes/base_link.STL
- added link kr4_5_schunk_left_link, mass 9.1881E-07; collision mesh filename=package://schunk_25nnb/meshes/left_link.STL; visual mesh filename=package://schunk_25nnb/meshes/left_link.STL
- added link kr4_5_schunk_right_link, mass 9.1881E-07; collision mesh filename=package://schunk_25nnb/meshes/right_link.STL; visual mesh filename=package://schunk_25nnb/meshes/right_link.STL
- added link kr4_5_tool0
Joints:
- removed joint kr3_disp__joint_base
- removed joint kr3_disp_flange-tool0
- removed joint kr3_disp_joint_a1
- removed joint kr3_disp_joint_a2
- removed joint kr3_disp_joint_a3
- removed joint kr3_disp_joint_a4
- removed joint kr3_disp_joint_a5
- removed joint kr3_disp_joint_a6
- removed joint kr3_disp_joint_a6-tool0
- removed joint kr3_pip__joint_base
- removed joint kr3_pip_flange-tool0
- removed joint kr3_pip_joint_a1
- removed joint kr3_pip_joint_a2
- removed joint kr3_pip_joint_a3
- removed joint kr3_pip_joint_a4
- removed joint kr3_pip_joint_a5
- removed joint kr3_pip_joint_a6
- removed joint kr3_pip_joint_a6-tool0
- removed joint kr3_pp1__joint_base
- removed joint kr3_pp1_flange-tool0
- removed joint kr3_pp1_joint_a1
- removed joint kr3_pp1_joint_a2
- removed joint kr3_pp1_joint_a3
- removed joint kr3_pp1_joint_a4
- removed joint kr3_pp1_joint_a5
- removed joint kr3_pp1_joint_a6
- removed joint kr3_pp1_joint_a6-tool0
- removed joint kr3_pp1_schunk_base_joint
- removed joint kr3_pp1_schunk_joint_left
- removed joint kr3_pp1_schunk_joint_right
- removed joint kr3_pp2__joint_base
- removed joint kr3_pp2_flange-tool0
- removed joint kr3_pp2_joint_a1
- removed joint kr3_pp2_joint_a2
- removed joint kr3_pp2_joint_a3
- removed joint kr3_pp2_joint_a4
- removed joint kr3_pp2_joint_a5
- removed joint kr3_pp2_joint_a6
- removed joint kr3_pp2_joint_a6-tool0
- removed joint kr3_pp2_schunk_base_joint
- removed joint kr3_pp2_schunk_joint_left
- removed joint kr3_pp2_schunk_joint_right
- removed joint kr4_pp3__joint_base
- removed joint kr4_pp3_joint_a1
- removed joint kr4_pp3_joint_a2
- removed joint kr4_pp3_joint_a3
- removed joint kr4_pp3_joint_a4
- removed joint kr4_pp3_joint_a5
- removed joint kr4_pp3_joint_a6
- removed joint kr4_pp3_joint_a6-tool0
- removed joint kr4_pp3_kr4_pp3_base_joint
- removed joint kr4_pp3_kr4_pp3_joint_left
- removed joint kr4_pp3_kr4_pp3_joint_right
- added joint kr3_1__joint_base: type fixed, parent base, child kr3_1_base_link, origin xyz=0 -0.5 1 rpy=0 0 0
- added joint kr3_1_flange-tool0: type fixed, parent kr3_1_flange, child kr3_1_tool0, origin xyz=0 0 0 rpy=0 1.5707963267948966 0
- added joint kr3_1_joint_a1: type revolute, parent kr3_1_base_link, child kr3_1_link_1, origin xyz=0 0 0.345 rpy=0 0 0, axis 0 0 -1, limit lower=-2.9670597283903604 upper=2.9670597283903604 effort=100 velocity=9.250245035569947
- added joint kr3_1_joint_a2: type revolute, parent kr3_1_link_1, child kr3_1_link_2, origin xyz=0.020 0 0 rpy=0 -1 0, axis 0 1 0, limit lower=-2.9670597283903604 upper=0.8726646259971648 effort=100 velocity=9.232791743050003
- added joint kr3_1_joint_a3: type revolute, parent kr3_1_link_2, child kr3_1_link_3, origin xyz=0.260 0 0 rpy=0 0 0, axis 0 1 0, limit lower=-1.9198621771937625 upper=2.705260340591211 effort=100 velocity=9.389871375729493
- added joint kr3_1_joint_a4: type revolute, parent kr3_1_link_3, child kr3_1_link_4, origin xyz=0 0 0.020 rpy=0 0 0, axis -1 0 0, limit lower=-3.0543261909900767 upper=3.0543261909900767 effort=100 velocity=10.471975511965978
- added joint kr3_1_joint_a5: type revolute, parent kr3_1_link_4, child kr3_1_link_5, origin xyz=0.260 0 0 rpy=0 0 0, axis 0 1 0, limit lower=-2.0943951023931953 upper=2.0943951023931953 effort=100 velocity=10.471975511965978
- added joint kr3_1_joint_a6: type revolute, parent kr3_1_link_5, child kr3_1_link_6, origin xyz=0.075 0 0 rpy=0 0 0, axis -1 0 0, limit lower=-6.1086523819801535 upper=6.1086523819801535 effort=100 velocity=13.962634015954636
- added joint kr3_1_joint_a6-tool0: type fixed, parent kr3_1_link_6, child kr3_1_flange, origin xyz=0 0 0 rpy=0 0 0
- added joint kr3_1_schunk_base_joint: type fixed, parent kr3_1_tool0, child kr3_1_schunk_base_link, origin xyz=0 0 0 rpy=0 0 -1.5707963267948966
- added joint kr3_1_schunk_joint_left: type prismatic, parent kr3_1_schunk_base_link, child kr3_1_schunk_left_link, origin xyz=0 -8.2944E-05 0.08056 rpy=1.5708 0 -3.1416, axis 1 0 0, limit lower=-0.0047 upper=1E-05 effort=20.0001 velocity=2.00001
- added joint kr3_1_schunk_joint_right: type prismatic, parent kr3_1_schunk_base_link, child kr3_1_schunk_right_link, origin xyz=0 -8.2944E-05 0.08056 rpy=1.5708 0 0, axis 1 0 0, limit lower=-0.0047 upper=1E-05 effort=20.00001 velocity=2.00001
- added joint kr3_2__joint_base: type fixed, parent base, child kr3_2_base_link, origin xyz=0 0.5 1 rpy=0 0 0
- added joint kr3_2_flange-tool0: type fixed, parent kr3_2_flange, child kr3_2_tool0, origin xyz=0 0 0 rpy=0 1.5707963267948966 0
- added joint kr3_2_joint_a1: type revolute, parent kr3_2_base_link, child kr3_2_link_1, origin xyz=0 0 0.345 rpy=0 0 0, axis 0 0 -1, limit lower=-2.9670597283903604 upper=2.9670597283903604 effort=100 velocity=9.250245035569947
- added joint kr3_2_joint_a2: type revolute, parent kr3_2_link_1, child kr3_2_link_2, origin xyz=0.020 0 0 rpy=0 -1 0, axis 0 1 0, limit lower=-2.9670597283903604 upper=0.8726646259971648 effort=100 velocity=9.232791743050003
- added joint kr3_2_joint_a3: type revolute, parent kr3_2_link_2, child kr3_2_link_3, origin xyz=0.260 0 0 rpy=0 0 0, axis 0 1 0, limit lower=-1.9198621771937625 upper=2.705260340591211 effort=100 velocity=9.389871375729493
- added joint kr3_2_joint_a4: type revolute, parent kr3_2_link_3, child kr3_2_link_4, origin xyz=0 0 0.020 rpy=0 0 0, axis -1 0 0, limit lower=-3.0543261909900767 upper=3.0543261909900767 effort=100 velocity=10.471975511965978
- added joint kr3_2_joint_a5: type revolute, parent kr3_2_link_4, child kr3_2_link_5, origin xyz=0.260 0 0 rpy=0 0 0, axis 0 1 0, limit lower=-2.0943951023931953 upper=2.0943951023931953 effort=100 velocity=10.471975511965978
- added joint kr3_2_joint_a6: type revolute, parent kr3_2_link_5, child kr3_2_link_6, origin xyz=0.075 0 0 rpy=0 0 0, axis -1 0 0, limit lower=-6.1086523819801535 upper=6.1086523819801535 effort=100 velocity=13.962634015954636
- added joint kr3_2_joint_a6-tool0: type fixed, parent kr3_2_link_6, child kr3_2_flange, origin xyz=0 0 0 rpy=0 0 0
- added joint kr3_2_schunk_base_joint: type fixed, parent kr3_2_tool0, child kr3_2_schunk_base_link, origin xyz=0 0 0 rpy=0 0 -1.5707963267948966
- added joint kr3_2_schunk_joint_left: type prismatic, parent kr3_2_schunk_base_link, child kr3_2_schunk_left_link, origin xyz=0 -8.2944E-05 0.08056 rpy=1.5708 0 -3.1416, axis 1 0 0, limit lower=-0.0047 upper=1E-05 effort=20.0001 velocity=2.00001
- added joint kr3_2_schunk_joint_right: type prismatic, parent kr3_2_schunk_base_link, child kr3_2_schunk_right_link, origin xyz=0 -8.2944E-05 0.08056 rpy=1.5708 0 0, axis 1 0 0, limit lower=-0.0047 upper=1E-05 effort=20.00001 velocity=2.00001
- added joint kr3_3__joint_base: type fixed, parent base, child kr3_3_base_link, origin xyz=1.9 -0.5 1 rpy=0 0 -3.141592653589793
- added joint kr3_3_flange-tool0: type fixed, parent kr3_3_flange, child kr3_3_tool0, origin xyz=0 0 0 rpy=0 1.5707963267948966 0
- added joint kr3_3_joint_a1: type revolute, parent kr3_3_base_link, child kr3_3_link_1, origin xyz=0 0 0.345 rpy=0 0 0, axis 0 0 -1, limit lower=-2.9670597283903604 upper=2.9670597283903604 effort=100 velocity=9.250245035569947
- added joint kr3_3_joint_a2: type revolute, parent kr3_3_link_1, child kr3_3_link_2, origin xyz=0.020 0 0 rpy=0 -1 0, axis 0 1 0, limit lower=-2.9670597283903604 upper=0.8726646259971648 effort=100 velocity=9.232791743050003
- added joint kr3_3_joint_a3: type revolute, parent kr3_3_link_2, child kr3_3_link_3, origin xyz=0.260 0 0 rpy=0 0 0, axis 0 1 0, limit lower=-1.9198621771937625 upper=2.705260340591211 effort=100 velocity=9.389871375729493
- added joint kr3_3_joint_a4: type revolute, parent kr3_3_link_3, child kr3_3_link_4, origin xyz=0 0 0.020 rpy=0 0 0, axis -1 0 0, limit lower=-3.0543261909900767 upper=3.0543261909900767 effort=100 velocity=10.471975511965978
- added joint kr3_3_joint_a5: type revolute, parent kr3_3_link_4, child kr3_3_link_5, origin xyz=0.260 0 0 rpy=0 0 0, axis 0 1 0, limit lower=-2.0943951023931953 upper=2.0943951023931953 effort=100 velocity=10.471975511965978
- added joint kr3_3_joint_a6: type revolute, parent kr3_3_link_5, child kr3_3_link_6, origin xyz=0.075 0 0 rpy=0 0 0, axis -1 0 0, limit lower=-6.1086523819801535 upper=6.1086523819801535 effort=100 velocity=13.962634015954636
- added joint kr3_3_joint_a6-tool0: type fixed, parent kr3_3_link_6, child kr3_3_flange, origin xyz=0 0 0 rpy=0 0 0
- added joint kr3_3_pip_base_joint: type fixed, parent kr3_3_tool0, child kr3_3_pip_base_link, origin xyz=0 0 0 rpy=0 3.141592653589793 -1.5707963267948966
- added joint kr3_4__joint_base: type fixed, parent base, child kr3_4_base_link, origin xyz=1.9 0.5 1 rpy=0 0 -3.141592653589793
- added joint kr3_4_disp_base_joint: type fixed, parent kr3_4_tool0, child kr3_4_disp_base_link, origin xyz=0 0 0 rpy=0 3.141592653589793 -1.5707963267948966
- added joint kr3_4_flange-tool0: type fixed, parent kr3_4_flange, child kr3_4_tool0, origin xyz=0 0 0 rpy=0 1.5707963267948966 0
- added joint kr3_4_joint_a1: type revolute, parent kr3_4_base_link, child kr3_4_link_1, origin xyz=0 0 0.345 rpy=0 0 0, axis 0 0 -1, limit lower=-2.9670597283903604 upper=2.9670597283903604 effort=100 velocity=9.250245035569947
- added joint kr3_4_joint_a2: type revolute, parent kr3_4_link_1, child kr3_4_link_2, origin xyz=0.020 0 0 rpy=0 -1 0, axis 0 1 0, limit lower=-2.9670597283903604 upper=0.8726646259971648 effort=100 velocity=9.232791743050003
- added joint kr3_4_joint_a3: type revolute, parent kr3_4_link_2, child kr3_4_link_3, origin xyz=0.260 0 0 rpy=0 0 0, axis 0 1 0, limit lower=-1.9198621771937625 upper=2.705260340591211 effort=100 velocity=9.389871375729493
- added joint kr3_4_joint_a4: type revolute, parent kr3_4_link_3, child kr3_4_link_4, origin xyz=0 0 0.020 rpy=0 0 0, axis -1 0 0, limit lower=-3.0543261909900767 upper=3.0543261909900767 effort=100 velocity=10.471975511965978
- added joint kr3_4_joint_a5: type revolute, parent kr3_4_link_4, child kr3_4_link_5, origin xyz=0.260 0 0 rpy=0 0 0, axis 0 1 0, limit lower=-2.0943951023931953 upper=2.0943951023931953 effort=100 velocity=10.471975511965978
- added joint kr3_4_joint_a6: type revolute, parent kr3_4_link_5, child kr3_4_link_6, origin xyz=0.075 0 0 rpy=0 0 0, axis -1 0 0, limit lower=-6.1086523819801535 upper=6.1086523819801535 effort=100 velocity=13.962634015954636
- added joint kr3_4_joint_a6-tool0: type fixed, parent kr3_4_link_6, child kr3_4_flange, origin xyz=0 0 0 rpy=0 0 0
- added joint kr4_5__joint_base: type fixed, parent base, child kr4_5_base_link, origin xyz=1.9 -1.5 1 rpy=0 0 -3.141592653589793
- added joint kr4_5_joint_a1: type revolute, parent kr4_5_base_link, child kr4_5_link_1, origin xyz=0 0 0.33 rpy=0 0 0, axis 0 0 -1, limit lower=-2.9670597283903604 upper=2.9670597283903604 effort=100 velocity=9.250245035569947
- added joint kr4_5_joint_a2: type revolute, parent kr4_5_link_1, child kr4_5_link_2, origin xyz=0.020 0 0 rpy=0 -1 0, axis 0 1 0, limit lower=-3.4033920413889427 upper=0.6981317007977318 effort=100 velocity=9.232791743050003
- added joint kr4_5_joint_a3: type revolute, parent kr4_5_link_2, child kr4_5_link_3, origin xyz=0.290 0 0 rpy=0 0 0, axis 0 1 0, limit lower=-2.007128639793479 upper=2.6179938779914944 effort=100 velocity=9.389871375729493
- added joint kr4_5_joint_a4: type revolute, parent kr4_5_link_3, child kr4_5_link_4, origin xyz=0.310 0 0.020 rpy=0 0 0, axis -1 0 0, limit lower=-3.2288591161895095 upper=3.2288591161895095 effort=100 velocity=10.471975511965978
- added joint kr4_5_joint_a5: type revolute, parent kr4_5_link_4, child kr4_5_link_5, origin xyz=0 0 0 rpy=0 0 0, axis 0 1 0, limit lower=-2.0943951023931953 upper=2.0943951023931953 effort=100 velocity=10.471975511965978
- added joint kr4_5_joint_a6: type revolute, parent kr4_5_link_5, child kr4_5_link_6, origin xyz=0.075 0 0 rpy=0 0 0, axis -1 0 0, limit lower=-6.1086523819801535 upper=6.1086523819801535 effort=100 velocity=13.962634015954636
- added joint kr4_5_joint_a6-tool0: type fixed, parent kr4_5_link_6, child kr4_5_tool0, origin xyz=0 0 0 rpy=0 1.5707963267948966 0
- added joint kr4_5_schunk_base_joint: type fixed, parent kr4_5_tool0, child kr4_5_schunk_base_link, origin xyz=0 0 0 rpy=0 0 -1.5707963267948966
- added joint kr4_5_schunk_joint_left: type prismatic, parent kr4_5_schunk_base_link, child kr4_5_schunk_left_link, origin xyz=0 -8.2944E-05 0.08056 rpy=1.5708 0 -3.1416, axis 1 0 0, limit lower=-0.0047 upper=1E-05 effort=20.0001 velocity=2.00001
- added joint kr4_5_schunk_joint_right: type prismatic, parent kr4_5_schunk_base_link, child kr4_5_schunk_right_link, origin xyz=0 -8.2944E-05 0.08056 rpy=1.5708 0 0, axis 1 0 0, limit lower=-0.0047 upper=1E-05 effort=20.00001 velocity=2.00001
