Commit message: Added pipette and dispenser to xacro macro and xacro tools

File: src/kuka_multiple_arms/robot_description/kuka_multiple_arms.xacro (robot description, xacro)
@@ -2,20 +2,20 @@
 <robot name="kuka_multiple_arms" xmlns:xacro="http://ros.org/wiki/xacro">
     <!-- add arms names prefixes -->
-    <xacro:arg name="arm_id_1" default="kr3_pp1_" />
-    <xacro:arg name="arm_id_2" default="kr3_pp2_" />
-    <xacro:arg name="arm_id_3" default="kr3_disp_" />
-    <xacro:arg name="arm_id_4" default="kr3_pip_" />
-    <xacro:arg name="arm_id_5" default="kr4_pp3_" />
+    <xacro:arg name="arm_id_1" default="kr3_1_" />
+    <xacro:arg name="arm_id_2" default="kr3_2_" />
+    <xacro:arg name="arm_id_3" default="kr3_3_" />
+    <xacro:arg name="arm_id_4" default="kr3_4_" />
+    <xacro:arg name="arm_id_5" default="kr4_5_" />
     <!-- add gripper names prefixes -->
     <xacro:arg name="hand_id_1" default="schunk_" />
     <xacro:arg name="hand_id_2" default="schunk_" />
-    <xacro:arg name="hand_id_3" default="kr3_disp_" />
-    <xacro:arg name="hand_id_4" default="kr3_pip_" />
-    <xacro:arg name="hand_id_5" default="kr4_pp3_" />
+    <xacro:arg name="hand_id_3" default="pip_" />
+    <xacro:arg name="hand_id_4" default="disp_" />
+    <xacro:arg name="hand_id_5" default="schunk_" />
     <!-- load arm/hand models and utils (which adds the robot inertia tags to be Gazebo-simulation ready) -->
-    <!-- <xacro:include filename="$(find kuka_kr3_support)/urdf/kr3r540_macro_v2.xacro"/> -->
     <xacro:include filename="$(find kuka_kr3_support)/urdf/kr3r540_macro_v2.xacro"/>
     <xacro:include filename="$(find kuka_kr4_support)/urdf/kr4r600_macro_v2.xacro"/>
-    <xacro:include filename="$(find schunk_25nnb)/urdf/schunk_25nnb_macro.xacro"/>
+    <!-- <xacro:include filename="$(find schunk_25nnb)/urdf/schunk_25nnb_macro.xacro"/> -->
+    <xacro:include filename="$(find kuka_kr3_support)/urdf/tools_macro.xacro"/>
     <link name="world"/>
     <!-- box shaped table as base for kukas -->
@@ -55,12 +55,10 @@
     <!-- ROBOT 3 with gripper -->
     <xacro:kuka_kr3r540 prefix="$(arg arm_id_3)" connected_to="base"  xyz="1.9 -0.5 1"  rpy="0 0 ${-pi}"/>
-    <!-- <xacro:kuka_gripper arm_id="$(arg arm_id_1)" rpy="0 0 ${-pi/4}" connected_to="$(arg arm_id_1)_flange" /> -->
+    <xacro:pipette prefix="$(arg arm_id_3)$(arg hand_id_3)"  rpy="0 ${pi} ${-pi/2}" connected_to="$(arg arm_id_3)tool0" />
     <!-- ROBOT 4 with gripper -->
     <xacro:kuka_kr3r540 prefix="$(arg arm_id_4)" connected_to="base"  xyz="1.9 0.5 1"  rpy="0 0 ${-pi}"/>
-    <!-- <xacro:kuka_gripper arm_id="$(arg arm_id_2)" rpy="0 0 ${-pi/4}" connected_to="$(arg arm_id_2)_flange" /> -->
+    <xacro:dispenser prefix="$(arg arm_id_4)$(arg hand_id_4)"  rpy="0 ${pi} ${-pi/2}" connected_to="$(arg arm_id_4)tool0" />
     <!-- ROBOT 5 with gripper -->
     <xacro:kuka_kr4r600 prefix="$(arg arm_id_5)" connected_to="base"  xyz="1.9 -1.5 1"  rpy="0 0 ${-pi}"/>
     <xacro:schunk_25nnb prefix="$(arg arm_id_5)$(arg hand_id_5)"  rpy="0 0 ${-pi/2}" connected_to="$(arg arm_id_5)tool0" />
-    <!-- <xacro:franka_arm arm_id="$(arg arm_id_2)" connected_to="base" xyz="0 0.5 1" gazebo="true" safety_distance="0.03" joint_limits="${xacro.load_yaml('$(find franka_description)/robots/panda/joint_limits.yaml')}"/>
-    <xacro:franka_hand arm_id="$(arg arm_id_2)" rpy="0 0 ${-pi/4}" connected_to="$(arg arm_id_2)_link8" gazebo="true" safety_distance="0.03" /> -->
 </robot>
