Commit message: gripper orientation

File: src/kuka_kr3_support/urdf/tools_macro.xacro (robot description, xacro)
@@ -92,6 +92,6 @@
         type="prismatic">
         <origin
-          xyz="0 -8.2944E-05 0.08056"
-          rpy="1.5708 0 -3.1416" />
+          xyz="0.076 -8.2944E-05 0"
+          rpy="1.5708 0 0" />
         <parent
           link="${prefix}base_link" />
@@ -150,5 +150,5 @@
         type="prismatic">
         <origin
-          xyz="0 -8.2944E-05 0.08056"
+          xyz="0.076 -8.2944E-05 0"
           rpy="1.5708 0 0" />
         <parent

File: src/kuka_multiple_arms/robot_description/kuka_multiple_arms.urdf (robot description, URDF)
Before this commit: robot kuka_multiple_arms, 57 links, 56 joints
Joints:
- joint kr3_1_schunk_base_joint: origin xyz=0 0 0 rpy=0 0 -1.5707963267948966 -> xyz=0 0 0 rpy=0 -1.5707963267948966 0
- joint kr3_1_schunk_joint_left: origin xyz=0 -8.2944E-05 0.08056 rpy=1.5708 0 -3.1416 -> xyz=0.076 -8.2944E-05 0 rpy=1.5708 0 0
- joint kr3_1_schunk_joint_right: origin xyz=0 -8.2944E-05 0.08056 rpy=1.5708 0 0 -> xyz=0.076 -8.2944E-05 0 rpy=1.5708 0 0
- joint kr3_2_schunk_base_joint: origin xyz=0 0 0 rpy=0 0 -1.5707963267948966 -> xyz=0 0 0 rpy=0 -1.5707963267948966 0
- joint kr3_2_schunk_joint_left: origin xyz=0 -8.2944E-05 0.08056 rpy=1.5708 0 -3.1416 -> xyz=0.076 -8.2944E-05 0 rpy=1.5708 0 0
- joint kr3_2_schunk_joint_right: origin xyz=0 -8.2944E-05 0.08056 rpy=1.5708 0 0 -> xyz=0.076 -8.2944E-05 0 rpy=1.5708 0 0
- joint kr4_5_schunk_base_joint: origin xyz=0 0 0 rpy=0 0 -1.5707963267948966 -> xyz=0 0 0 rpy=0 -1.5707963267948966 0
- joint kr4_5_schunk_joint_left: origin xyz=0 -8.2944E-05 0.08056 rpy=1.5708 0 -3.1416 -> xyz=0.076 -8.2944E-05 0 rpy=1.5708 0 0
- joint kr4_5_schunk_joint_right: origin xyz=0 -8.2944E-05 0.08056 rpy=1.5708 0 0 -> xyz=0.076 -8.2944E-05 0 rpy=1.5708 0 0

File: src/kuka_multiple_arms/robot_description/kuka_multiple_arms.xacro (robot description, xacro)
@@ -57,8 +57,8 @@
     <!-- ROBOT 1 with gripper -->
     <xacro:kuka_kr3r540 prefix="$(arg arm_id_1)" connected_to="base"  xyz="0.171 -1.16645 0"  rpy="0 0 ${pi/2}"/>
-    <xacro:schunk_25nnb prefix="$(arg arm_id_1)$(arg hand_id_1)"  rpy="0 0 ${-pi/2}" connected_to="$(arg arm_id_1)tool0" />
+    <xacro:schunk_25nnb prefix="$(arg arm_id_1)$(arg hand_id_1)"  rpy="0 ${-pi/2} 0" connected_to="$(arg arm_id_1)tool0" />
     <!-- ROBOT 2 with gripper -->
     <xacro:kuka_kr3r540 prefix="$(arg arm_id_2)" connected_to="base"  xyz="0.729 -1.16645 0" rpy="0 0 ${pi/2}" />
-    <xacro:schunk_25nnb prefix="$(arg arm_id_2)$(arg hand_id_2)"  rpy="0 0 ${-pi/2}" connected_to="$(arg arm_id_2)tool0" />
+    <xacro:schunk_25nnb prefix="$(arg arm_id_2)$(arg hand_id_2)"  rpy="0 ${-pi/2} 0" connected_to="$(arg arm_id_2)tool0" />
     <!-- ROBOT 3 with gripper -->
     <xacro:kuka_kr3r540 prefix="$(arg arm_id_3)" connected_to="base"  xyz="0.171 -0.20714 0"  rpy="0 0 ${-pi/2}"/>
@@ -69,4 +69,4 @@
     <!-- ROBOT 5 with gripper -->
     <xacro:kuka_kr4r600 prefix="$(arg arm_id_5)" connected_to="base"  xyz="1.37418 -0.20714 0"  rpy="0 0 ${-pi/2}"/>
-    <xacro:schunk_25nnb prefix="$(arg arm_id_5)$(arg hand_id_5)"  rpy="0 0 ${-pi/2}" connected_to="$(arg arm_id_5)tool0" />
+    <xacro:schunk_25nnb prefix="$(arg arm_id_5)$(arg hand_id_5)"  rpy="0 ${-pi/2} 0" connected_to="$(arg arm_id_5)tool0" />
 </robot>

File: src/schunk_25nnb/urdf/schunk_25nnb.urdf (robot description, URDF)
Before this commit: robot schunk_25nnb, 3 links, 2 joints
Links:
- link base_link: mass 3.0843E-05 -> 0.03199945156995
- link left_link: mass 0.016862 -> 0.028312
- link right_link: mass 0.016862 -> 0.028333
Joints:
- joint joint_left: axis 1 0 0 -> 0 1 0; limit lower=-0.0047 upper=1E-05 effort=20 velocity=2 -> lower=-0.003 upper=0 effort=40 velocity=2; origin xyz=0 -8.2944E-05 0.08056 rpy=1.5708 0 -3.1416 -> xyz=0 0 0 rpy=0 0 0
- joint joint_right: axis 1 0 0 -> 0 1 0; limit lower=-0.0047 upper=1E-05 effort=20 velocity=2 -> lower=-0.003 upper=0 effort=40 velocity=2; origin xyz=0 -8.2944E-05 0.08056 rpy=1.5708 0 0 -> xyz=0 0 0 rpy=0 0 0
