Commit message: Kr3r540 usd gripper

File: src/kuka_kr3_support/urdf/kr3r540_v4.urdf (robot description, URDF)
Before this commit: robot kuka_kr3r540, 13 links, 12 joints
Joints:
- joint joint_left: origin xyz=0 -8.2944E-05 0.08056 rpy=1.5708 0 3.1416 -> xyz=0 -8.2944E-05 0.08056 rpy=0 0 0
- joint joint_right: origin xyz=0 -8.2944E-05 0.08056 rpy=1.5708 0 0 -> xyz=0 -8.2944E-05 0.08056 rpy=0 0 0
