Commit message: multiple config file

File: src/kuka_config_multiple/config/gazebo_kuka_multiple_arms.urdf (robot description, URDF)
Before this commit: robot kuka_multiple_arms, 57 links, 56 joints
Joints:
- joint kr3_1_schunk_base_joint: origin xyz=0 0 0 rpy=0 0 -1.5707963267948966 -> xyz=0 0 0 rpy=0 -1.5707963267948966 0
- joint kr3_1_schunk_joint_left: origin xyz=0 -8.2944E-05 0.08056 rpy=1.5708 0 -3.1416 -> xyz=0.076 -8.2944E-05 0 rpy=1.5708 0 0
- joint kr3_1_schunk_joint_right: origin xyz=0 -8.2944E-05 0.08056 rpy=1.5708 0 0 -> xyz=0.076 -8.2944E-05 0 rpy=1.5708 0 0
- joint kr3_2_schunk_base_joint: origin xyz=0 0 0 rpy=0 0 -1.5707963267948966 -> xyz=0 0 0 rpy=0 -1.5707963267948966 0
- joint kr3_2_schunk_joint_left: origin xyz=0 -8.2944E-05 0.08056 rpy=1.5708 0 -3.1416 -> xyz=0.076 -8.2944E-05 0 rpy=1.5708 0 0
- joint kr3_2_schunk_joint_right: origin xyz=0 -8.2944E-05 0.08056 rpy=1.5708 0 0 -> xyz=0.076 -8.2944E-05 0 rpy=1.5708 0 0
- joint kr4_5_schunk_base_joint: origin xyz=0 0 0 rpy=0 0 -1.5707963267948966 -> xyz=0 0 0 rpy=0 -1.5707963267948966 0
- joint kr4_5_schunk_joint_left: origin xyz=0 -8.2944E-05 0.08056 rpy=1.5708 0 -3.1416 -> xyz=0.076 -8.2944E-05 0 rpy=1.5708 0 0
- joint kr4_5_schunk_joint_right: origin xyz=0 -8.2944E-05 0.08056 rpy=1.5708 0 0 -> xyz=0.076 -8.2944E-05 0 rpy=1.5708 0 0

Commit message: Old gripper

File: src/kuka_config_multiple/config/gazebo_kuka_multiple_arms.urdf (robot description, URDF)
Before this commit: robot kuka_multiple_arms, 57 links, 56 joints
Joints:
- joint kr3_1_schunk_base_joint: origin xyz=0 0 0 rpy=0 -1.5707963267948966 0 -> xyz=0 0 0 rpy=0 0 -1.5707963267948966
- joint kr3_1_schunk_joint_left: origin xyz=0.076 -8.2944E-05 0 rpy=1.5708 0 0 -> xyz=0 -8.2944E-05 0.08056 rpy=1.5708 0 -3.1416
- joint kr3_1_schunk_joint_right: origin xyz=0.076 -8.2944E-05 0 rpy=1.5708 0 0 -> xyz=0 -8.2944E-05 0.08056 rpy=1.5708 0 0
- joint kr3_2_schunk_base_joint: origin xyz=0 0 0 rpy=0 -1.5707963267948966 0 -> xyz=0 0 0 rpy=0 0 -1.5707963267948966
- joint kr3_2_schunk_joint_left: origin xyz=0.076 -8.2944E-05 0 rpy=1.5708 0 0 -> xyz=0 -8.2944E-05 0.08056 rpy=1.5708 0 -3.1416
- joint kr3_2_schunk_joint_right: origin xyz=0.076 -8.2944E-05 0 rpy=1.5708 0 0 -> xyz=0 -8.2944E-05 0.08056 rpy=1.5708 0 0
- joint kr4_5_schunk_base_joint: origin xyz=0 0 0 rpy=0 -1.5707963267948966 0 -> xyz=0 0 0 rpy=0 0 -1.5707963267948966
- joint kr4_5_schunk_joint_left: origin xyz=0.076 -8.2944E-05 0 rpy=1.5708 0 0 -> xyz=0 -8.2944E-05 0.08056 rpy=1.5708 0 -3.1416
- joint kr4_5_schunk_joint_right: origin xyz=0.076 -8.2944E-05 0 rpy=1.5708 0 0 -> xyz=0 -8.2944E-05 0.08056 rpy=1.5708 0 0

File: src/kuka_kr3_support/urdf/tools_macro.xacro (robot description, xacro)
@@ -92,6 +92,6 @@
         type="prismatic">
         <origin
-          xyz="0.076 -8.2944E-05 0"
-          rpy="1.5708 0 0" />
+          xyz="0 -8.2944E-05 0.08056"
+          rpy="1.5708 0 -3.1416" />
         <parent
           link="${prefix}base_link" />
@@ -150,5 +150,5 @@
         type="prismatic">
         <origin
-          xyz="0.076 -8.2944E-05 0"
+          xyz="0 -8.2944E-05 0.08056"
           rpy="1.5708 0 0" />
         <parent

File: src/kuka_multiple_arms/robot_description/kuka_multiple_arms.urdf (robot description, URDF)
Before this commit: robot kuka_multiple_arms, 57 links, 56 joints
Joints:
- joint kr3_1_schunk_base_joint: origin xyz=0 0 0 rpy=0 -1.5707963267948966 0 -> xyz=0 0 0 rpy=0 0 -1.5707963267948966
- joint kr3_1_schunk_joint_left: origin xyz=0.076 -8.2944E-05 0 rpy=1.5708 0 0 -> xyz=0 -8.2944E-05 0.08056 rpy=1.5708 0 -3.1416
- joint kr3_1_schunk_joint_right: origin xyz=0.076 -8.2944E-05 0 rpy=1.5708 0 0 -> xyz=0 -8.2944E-05 0.08056 rpy=1.5708 0 0
- joint kr3_2_schunk_base_joint: origin xyz=0 0 0 rpy=0 -1.5707963267948966 0 -> xyz=0 0 0 rpy=0 0 -1.5707963267948966
- joint kr3_2_schunk_joint_left: origin xyz=0.076 -8.2944E-05 0 rpy=1.5708 0 0 -> xyz=0 -8.2944E-05 0.08056 rpy=1.5708 0 -3.1416
- joint kr3_2_schunk_joint_right: origin xyz=0.076 -8.2944E-05 0 rpy=1.5708 0 0 -> xyz=0 -8.2944E-05 0.08056 rpy=1.5708 0 0
- joint kr4_5_schunk_base_joint: origin xyz=0 0 0 rpy=0 -1.5707963267948966 0 -> xyz=0 0 0 rpy=0 0 -1.5707963267948966
- joint kr4_5_schunk_joint_left: origin xyz=0.076 -8.2944E-05 0 rpy=1.5708 0 0 -> xyz=0 -8.2944E-05 0.08056 rpy=1.5708 0 -3.1416
- joint kr4_5_schunk_joint_right: origin xyz=0.076 -8.2944E-05 0 rpy=1.5708 0 0 -> xyz=0 -8.2944E-05 0.08056 rpy=1.5708 0 0

File: src/schunk_25nnb/urdf/schunk_25nnb.urdf (robot description, URDF)
Before this commit: robot schunk_25nnb, 3 links, 2 joints
Links:
- link base_link: mass 0.03199945156995 -> 3.08428949350963E-05
- link left_link: mass 0.028312 -> 9.1881E-07
- link right_link: mass 0.028333 -> 9.1881E-07
Joints:
- joint joint_left: axis 0 1 0 -> 1 0 0; limit lower=-0.003 upper=0 effort=40 velocity=2 -> lower=-0.0047 upper=1E-05 effort=20 velocity=2; origin xyz=0 0 0 rpy=0 0 0 -> xyz=0 -8.2944E-05 0.08056 rpy=1.5708 0 -3.1416
- joint joint_right: axis 0 1 0 -> 1 0 0; limit lower=-0.003 upper=0 effort=40 velocity=2 -> lower=-0.0047 upper=1E-05 effort=20 velocity=2; origin xyz=0 0 0 rpy=0 0 0 -> xyz=0 -8.2944E-05 0.08056 rpy=1.5708 0 0

Commit message: new kuka multiple config

File: src/kuka_config_multiple/config/gazebo_kuka_multiple_arms.urdf (robot description, URDF)
Before this commit: robot kuka_multiple_arms, 57 links, 56 joints
Joints:
- joint kr3_1_schunk_base_joint: origin xyz=0 0 0 rpy=0 0 -1.5707963267948966 -> xyz=0 0 0 rpy=0 0 0
- joint kr3_2_schunk_base_joint: origin xyz=0 0 0 rpy=0 0 -1.5707963267948966 -> xyz=0 0 0 rpy=0 0 0
- joint kr4_5_schunk_base_joint: origin xyz=0 0 0 rpy=0 0 -1.5707963267948966 -> xyz=0 0 0 rpy=0 0 0
