Commit message: Added macro for schunk grippers

File: src/kuka_multiple_arms/robot_description/kuka_multiple_arms.urdf (robot description, URDF)
Before this commit: robot kuka_multiple_arms, 20 links, 19 joints
Links:
- added link kr3_disp_base_link; collision mesh filename=package://kuka_kr3_support/meshes/kr3r540/collision/base_li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; visual mesh filename=package://kuka_kr3_support/meshes/kr3r540/visual/base_link.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
- added link kr3_disp_flange
- added link kr3_disp_link_1; collision mesh filename=package://kuka_kr3_support/meshes/kr3r540/collision/link_1.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; visual mesh filename=package://kuka_kr3_support/meshes/kr3r540/visual/link_1.stl
- added link kr3_disp_link_2; collision mesh filename=package://kuka_kr3_support/meshes/kr3r540/collision/link_2.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; visual mesh filename=package://kuka_kr3_support/meshes/kr3r540/visual/link_2.stl
- added link kr3_disp_link_3; collision mesh filename=package://kuka_kr3_support/meshes/kr3r540/collision/link_3.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; visual mesh filename=package://kuka_kr3_support/meshes/kr3r540/visual/link_3.stl
- added link kr3_disp_link_4; collision mesh filename=package://kuka_kr3_support/meshes/kr3r540/collision/link_4.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; visual mesh filename=package://kuka_kr3_support/meshes/kr3r540/visual/link_4.stl
- added link kr3_disp_link_5; collision mesh filename=package://kuka_kr3_support/meshes/kr3r540/collision/link_5.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; visual mesh filename=package://kuka_kr3_support/meshes/kr3r540/visual/link_5.stl
- added link kr3_disp_link_6; collision mesh filename=package://kuka_kr3_support/meshes/kr3r540/collision/link_6.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; visual mesh filename=package://kuka_kr3_support/meshes/kr3r540/visual/link_6.stl
- added link kr3_disp_tool0
- added link kr3_pip_base_link; collision mesh filename=package://kuka_kr3_support/meshes/kr3r540/collision/base_li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; visual mesh filename=package://kuka_kr3_support/meshes/kr3r540/visual/base_link.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
- added link kr3_pip_flange
- added link kr3_pip_link_1; collision mesh filename=package://kuka_kr3_support/meshes/kr3r540/collision/link_1.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; visual mesh filename=package://kuka_kr3_support/meshes/kr3r540/visual/link_1.stl
- added link kr3_pip_link_2; collision mesh filename=package://kuka_kr3_support/meshes/kr3r540/collision/link_2.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; visual mesh filename=package://kuka_kr3_support/meshes/kr3r540/visual/link_2.stl
- added link kr3_pip_link_3; collision mesh filename=package://kuka_kr3_support/meshes/kr3r540/collision/link_3.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; visual mesh filename=package://kuka_kr3_support/meshes/kr3r540/visual/link_3.stl
- added link kr3_pip_link_4; collision mesh filename=package://kuka_kr3_support/meshes/kr3r540/collision/link_4.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; visual mesh filename=package://kuka_kr3_support/meshes/kr3r540/visual/link_4.stl
- added link kr3_pip_link_5; collision mesh filename=package://kuka_kr3_support/meshes/kr3r540/collision/link_5.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; visual mesh filename=package://kuka_kr3_support/meshes/kr3r540/visual/link_5.stl
- added link kr3_pip_link_6; collision mesh filename=package://kuka_kr3_support/meshes/kr3r540/collision/link_6.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; visual mesh filename=package://kuka_kr3_support/meshes/kr3r540/visual/link_6.stl
- added link kr3_pip_tool0
- added link kr3_pp1_schunk_base_link, mass 3.08428949350963E-05; collision mesh filename=package://schunk_25nnb/meshes/base_link.STL; visual mesh filename=package://schunk_25nnb/meshes/base_link.STL
- added link kr3_pp1_schunk_left_link, mass 9.1881E-07; collision mesh filename=package://schunk_25nnb/meshes/left_link.STL; visual mesh filename=package://schunk_25nnb/meshes/left_link.STL
- added link kr3_pp1_schunk_right_link, mass 9.1881E-07; collision mesh filename=package://schunk_25nnb/meshes/right_link.STL; visual mesh filename=package://schunk_25nnb/meshes/right_link.STL
- added link kr3_pp2_schunk_base_link, mass 3.08428949350963E-05; collision mesh filename=package://schunk_25nnb/meshes/base_link.STL; visual mesh filename=package://schunk_25nnb/meshes/base_link.STL
- added link kr3_pp2_schunk_left_link, mass 9.1881E-07; collision mesh filename=package://schunk_25nnb/meshes/left_link.STL; visual mesh filename=package://schunk_25nnb/meshes/left_link.STL
- added link kr3_pp2_schunk_right_link, mass 9.1881E-07; collision mesh filename=package://schunk_25nnb/meshes/right_link.STL; visual mesh filename=package://schunk_25nnb/meshes/right_link.STL
Joints:
- added joint kr3_disp__joint_base: type fixed, parent base, child kr3_disp_base_link, origin xyz=1.9 -0.5 1 rpy=0 0 -3.141592653589793
- added joint kr3_disp_flange-tool0: type fixed, parent kr3_disp_flange, child kr3_disp_tool0, origin xyz=0 0 0 rpy=0 1.5707963267948966 0
- added joint kr3_disp_joint_a1: type revolute, parent kr3_disp_base_link, child kr3_disp_link_1, origin xyz=0 0 0.345 rpy=0 0 0, axis 0 0 -1, limit lower=-2.9670597283903604 upper=2.9670597283903604 effort=0 velocity=9.250245035569947
- added joint kr3_disp_joint_a2: type revolute, parent kr3_disp_link_1, child kr3_disp_link_2, origin xyz=0.020 0 0 rpy=0 0 0, axis 0 1 0, limit lower=-2.9670597283903604 upper=0.8726646259971648 effort=0 velocity=9.232791743050003
- added joint kr3_disp_joint_a3: type revolute, parent kr3_disp_link_2, child kr3_disp_link_3, origin xyz=0.260 0 0 rpy=0 0 0, axis 0 1 0, limit lower=-1.9198621771937625 upper=2.705260340591211 effort=0 velocity=9.389871375729493
- added joint kr3_disp_joint_a4: type revolute, parent kr3_disp_link_3, child kr3_disp_link_4, origin xyz=0 0 0.020 rpy=0 0 0, axis -1 0 0, limit lower=-3.0543261909900767 upper=3.0543261909900767 effort=0 velocity=10.471975511965978
- added joint kr3_disp_joint_a5: type revolute, parent kr3_disp_link_4, child kr3_disp_link_5, origin xyz=0.260 0 0 rpy=0 0 0, axis 0 1 0, limit lower=-2.0943951023931953 upper=2.0943951023931953 effort=0 velocity=10.471975511965978
- added joint kr3_disp_joint_a6: type revolute, parent kr3_disp_link_5, child kr3_disp_link_6, origin xyz=0.075 0 0 rpy=0 0 0, axis -1 0 0, limit lower=-6.1086523819801535 upper=6.1086523819801535 effort=0 velocity=13.962634015954636
- added joint kr3_disp_joint_a6-tool0: type fixed, parent kr3_disp_link_6, child kr3_disp_flange, origin xyz=0 0 0 rpy=0 0 0
- added joint kr3_pip__joint_base: type fixed, parent base, child kr3_pip_base_link, origin xyz=1.9 0.5 1 rpy=0 0 -3.141592653589793
- added joint kr3_pip_flange-tool0: type fixed, parent kr3_pip_flange, child kr3_pip_tool0, origin xyz=0 0 0 rpy=0 1.5707963267948966 0
- added joint kr3_pip_joint_a1: type revolute, parent kr3_pip_base_link, child kr3_pip_link_1, origin xyz=0 0 0.345 rpy=0 0 0, axis 0 0 -1, limit lower=-2.9670597283903604 upper=2.9670597283903604 effort=0 velocity=9.250245035569947
- added joint kr3_pip_joint_a2: type revolute, parent kr3_pip_link_1, child kr3_pip_link_2, origin xyz=0.020 0 0 rpy=0 0 0, axis 0 1 0, limit lower=-2.9670597283903604 upper=0.8726646259971648 effort=0 velocity=9.232791743050003
- added joint kr3_pip_joint_a3: type revolute, parent kr3_pip_link_2, child kr3_pip_link_3, origin xyz=0.260 0 0 rpy=0 0 0, axis 0 1 0, limit lower=-1.9198621771937625 upper=2.705260340591211 effort=0 velocity=9.389871375729493
- added joint kr3_pip_joint_a4: type revolute, parent kr3_pip_link_3, child kr3_pip_link_4, origin xyz=0 0 0.020 rpy=0 0 0, axis -1 0 0, limit lower=-3.0543261909900767 upper=3.0543261909900767 effort=0 velocity=10.471975511965978
- added joint kr3_pip_joint_a5: type revolute, parent kr3_pip_link_4, child kr3_pip_link_5, origin xyz=0.260 0 0 rpy=0 0 0, axis 0 1 0, limit lower=-2.0943951023931953 upper=2.0943951023931953 effort=0 velocity=10.471975511965978
- added joint kr3_pip_joint_a6: type revolute, parent kr3_pip_link_5, child kr3_pip_link_6, origin xyz=0.075 0 0 rpy=0 0 0, axis -1 0 0, limit lower=-6.1086523819801535 upper=6.1086523819801535 effort=0 velocity=13.962634015954636
- added joint kr3_pip_joint_a6-tool0: type fixed, parent kr3_pip_link_6, child kr3_pip_flange, origin xyz=0 0 0 rpy=0 0 0
- added joint kr3_pp1_schunk_base_joint: type fixed, parent kr3_pp1_tool0, child kr3_pp1_schunk_base_link, origin xyz=0 0 0 rpy=0 0 -1.5707963267948966
- added joint kr3_pp1_schunk_joint_left: type prismatic, parent kr3_pp1_schunk_base_link, child kr3_pp1_schunk_left_link, origin xyz=0 -8.2944E-05 0.08056 rpy=1.5708 0 -3.1416, axis 1 0 0, limit lower=-0.0047 upper=1E-05 effort=20 velocity=2
- added joint kr3_pp1_schunk_joint_right: type prismatic, parent kr3_pp1_schunk_base_link, child kr3_pp1_schunk_right_link, origin xyz=0 -8.2944E-05 0.08056 rpy=1.5708 0 0, axis 1 0 0, limit lower=-0.0047 upper=1E-05 effort=20.00001 velocity=2.00001
- added joint kr3_pp2_schunk_base_joint: type fixed, parent kr3_pp2_tool0, child kr3_pp2_schunk_base_link, origin xyz=0 0 0 rpy=0 0 -1.5707963267948966
- added joint kr3_pp2_schunk_joint_left: type prismatic, parent kr3_pp2_schunk_base_link, child kr3_pp2_schunk_left_link, origin xyz=0 -8.2944E-05 0.08056 rpy=1.5708 0 -3.1416, axis 1 0 0, limit lower=-0.0047 upper=1E-05 effort=20 velocity=2
- added joint kr3_pp2_schunk_joint_right: type prismatic, parent kr3_pp2_schunk_base_link, child kr3_pp2_schunk_right_link, origin xyz=0 -8.2944E-05 0.08056 rpy=1.5708 0 0, axis 1 0 0, limit lower=-0.0047 upper=1E-05 effort=20.00001 velocity=2.00001

File: src/kuka_multiple_arms/robot_description/kuka_multiple_arms.xacro (robot description, xacro)
@@ -4,9 +4,17 @@
     <xacro:arg name="arm_id_1" default="kr3_pp1_" />
     <xacro:arg name="arm_id_2" default="kr3_pp2_" />
+    <xacro:arg name="arm_id_3" default="kr3_disp_" />
+    <xacro:arg name="arm_id_4" default="kr3_pip_" />
+    <!-- add gripper names prefixes -->
+    <xacro:arg name="hand_id_1" default="schunk_" />
+    <xacro:arg name="hand_id_2" default="schunk_" />
+    <xacro:arg name="hand_id_3" default="kr3_disp_" />
+    <xacro:arg name="hand_id_4" default="kr3_pip_" />
     <!-- load arm/hand models and utils (which adds the robot inertia tags to be Gazebo-simulation ready) -->
     <!-- <xacro:include filename="$(find kuka_kr3_support)/urdf/kr3r540_macro_v2.xacro"/> -->
     <xacro:include filename="$(find kuka_kr3_support)/urdf/kr3r540_macro_v2.xacro"/>
+    <xacro:include filename="$(find schunk_25nnb)/urdf/schunk_25nnb_macro.xacro"/>
     <link name="world"/>
-    <!-- box shaped table as base for the 2 Pandas -->
+    <!-- box shaped table as base for kukas -->
     <link name="base">
         <visual>
@@ -37,8 +45,14 @@
     </joint>
     <!-- ROBOT 1 with gripper -->
-    <xacro:kuka_kr3r540 prefix="$(arg arm_id_1)" connected_to="base"  xyz="0 -0.5 1"  />
+    <xacro:kuka_kr3r540 prefix="$(arg arm_id_1)" connected_to="base"  xyz="0 -0.5 1"  rpy="0 0 0"/>
+    <xacro:schunk_25nnb prefix="$(arg arm_id_1)$(arg hand_id_1)"  rpy="0 0 ${-pi/2}" connected_to="$(arg arm_id_1)tool0" />
+    <!-- ROBOT 2 with gripper -->
+    <xacro:kuka_kr3r540 prefix="$(arg arm_id_2)" connected_to="base"  xyz="0 0.5 1" rpy="0 0 0" />
+    <xacro:schunk_25nnb prefix="$(arg arm_id_2)$(arg hand_id_2)"  rpy="0 0 ${-pi/2}" connected_to="$(arg arm_id_2)tool0" />
+    <!-- ROBOT 3 with gripper -->
+    <xacro:kuka_kr3r540 prefix="$(arg arm_id_3)" connected_to="base"  xyz="1.9 -0.5 1"  rpy="0 0 ${-pi}"/>
     <!-- <xacro:kuka_gripper arm_id="$(arg arm_id_1)" rpy="0 0 ${-pi/4}" connected_to="$(arg arm_id_1)_flange" /> -->
-    <!-- ROBOT 2 with gripper -->
-    <xacro:kuka_kr3r540 prefix="$(arg arm_id_2)" connected_to="base"  xyz="0 0.5 1"  />
+    <!-- ROBOT 4 with gripper -->
+    <xacro:kuka_kr3r540 prefix="$(arg arm_id_4)" connected_to="base"  xyz="1.9 0.5 1"  rpy="0 0 ${-pi}"/>
     <!-- <xacro:kuka_gripper arm_id="$(arg arm_id_2)" rpy="0 0 ${-pi/4}" connected_to="$(arg arm_id_2)_flange" /> -->
     <!-- <xacro:franka_arm arm_id="$(arg arm_id_2)" connected_to="base" xyz="0 0.5 1" gazebo="true" safety_distance="0.03" joint_limits="${xacro.load_yaml('$(find franka_description)/robots/panda/joint_limits.yaml')}"/>

Commit message: Added kr4r600 xacro macro

File: src/kuka_multiple_arms/robot_description/kuka_multiple_arms.urdf (robot description, URDF)
Before this commit: robot kuka_multiple_arms, 44 links, 43 joints
Links:
- added link kr4_pp3_base_link; collision mesh filename=package://kuka_kr4_support/meshes/kr4r600/collision/base_li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; visual mesh filename=package://kuka_kr4_support/meshes/kr4r600/visual/base_link.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
- added link kr4_pp3_kr4_pp3_base_link, mass 3.08428949350963E-05; collision mesh filename=package://schunk_25nnb/meshes/base_link.STL; visual mesh filename=package://schunk_25nnb/meshes/base_link.STL
- added link kr4_pp3_kr4_pp3_left_link, mass 9.1881E-07; collision mesh filename=package://schunk_25nnb/meshes/left_link.STL; visual mesh filename=package://schunk_25nnb/meshes/left_link.STL
- added link kr4_pp3_kr4_pp3_right_link, mass 9.1881E-07; collision mesh filename=package://schunk_25nnb/meshes/right_link.STL; visual mesh filename=package://schunk_25nnb/meshes/right_link.STL
- added link kr4_pp3_link_1; collision mesh filename=package://kuka_kr4_support/meshes/kr4r600/collision/link_1.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; visual mesh filename=package://kuka_kr4_support/meshes/kr4r600/visual/link_1.stl
- added link kr4_pp3_link_2; collision mesh filename=package://kuka_kr4_support/meshes/kr4r600/collision/link_2.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; visual mesh filename=package://kuka_kr4_support/meshes/kr4r600/visual/link_2.stl
- added link kr4_pp3_link_3; collision mesh filename=package://kuka_kr4_support/meshes/kr4r600/collision/link_3.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; visual mesh filename=package://kuka_kr4_support/meshes/kr4r600/visual/link_3.stl
- added link kr4_pp3_link_4; collision mesh filename=package://kuka_kr4_support/meshes/kr4r600/collision/link_4.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; visual mesh filename=package://kuka_kr4_support/meshes/kr4r600/visual/link_4.stl
- added link kr4_pp3_link_5; collision mesh filename=package://kuka_kr4_support/meshes/kr4r600/collision/link_5.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; visual mesh filename=package://kuka_kr4_support/meshes/kr4r600/visual/link_5.stl
- added link kr4_pp3_link_6; collision mesh filename=package://kuka_kr4_support/meshes/kr4r600/collision/link_6.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; visual mesh filename=package://kuka_kr4_support/meshes/kr4r600/visual/link_6.stl
- added link kr4_pp3_tool0
Joints:
- added joint kr4_pp3__joint_base: type fixed, parent base, child kr4_pp3_base_link, origin xyz=1.9 -1.5 1 rpy=0 0 -3.141592653589793
- added joint kr4_pp3_joint_a1: type revolute, parent kr4_pp3_base_link, child kr4_pp3_link_1, origin xyz=0 0 0.33 rpy=0 0 0, axis 0 0 -1, limit lower=-2.9670597283903604 upper=2.9670597283903604 effort=0 velocity=9.250245035569947
- added joint kr4_pp3_joint_a2: type revolute, parent kr4_pp3_link_1, child kr4_pp3_link_2, origin xyz=0 0 0 rpy=0 0 0, axis 0 1 0, limit lower=-3.4033920413889427 upper=0.6981317007977318 effort=0 velocity=9.232791743050003
- added joint kr4_pp3_joint_a3: type revolute, parent kr4_pp3_link_2, child kr4_pp3_link_3, origin xyz=0.290 0 0 rpy=0 0 0, axis 0 1 0, limit lower=-2.007128639793479 upper=2.6179938779914944 effort=0 velocity=9.389871375729493
- added joint kr4_pp3_joint_a4: type revolute, parent kr4_pp3_link_3, child kr4_pp3_link_4, origin xyz=0.310 0 0.020 rpy=0 0 0, axis -1 0 0, limit lower=-3.2288591161895095 upper=3.2288591161895095 effort=0 velocity=10.471975511965978
- added joint kr4_pp3_joint_a5: type revolute, parent kr4_pp3_link_4, child kr4_pp3_link_5, origin xyz=0 0 0 rpy=0 0 0, axis 0 1 0, limit lower=-2.0943951023931953 upper=2.0943951023931953 effort=0 velocity=10.471975511965978
- added joint kr4_pp3_joint_a6: type revolute, parent kr4_pp3_link_5, child kr4_pp3_link_6, origin xyz=0.075 0 0 rpy=0 0 0, axis -1 0 0, limit lower=-6.1086523819801535 upper=6.1086523819801535 effort=0 velocity=13.962634015954636
- added joint kr4_pp3_joint_a6-tool0: type fixed, parent kr4_pp3_link_6, child kr4_pp3_tool0, origin xyz=0 0 0 rpy=0 1.5707963267948966 0
- added joint kr4_pp3_kr4_pp3_base_joint: type fixed, parent kr4_pp3_tool0, child kr4_pp3_kr4_pp3_base_link, origin xyz=0 0 0 rpy=0 0 -1.5707963267948966
- added joint kr4_pp3_kr4_pp3_joint_left: type prismatic, parent kr4_pp3_kr4_pp3_base_link, child kr4_pp3_kr4_pp3_left_link, origin xyz=0 -8.2944E-05 0.08056 rpy=1.5708 0 -3.1416, axis 1 0 0, limit lower=-0.0047 upper=1E-05 effort=20 velocity=2
- added joint kr4_pp3_kr4_pp3_joint_right: type prismatic, parent kr4_pp3_kr4_pp3_base_link, child kr4_pp3_kr4_pp3_right_link, origin xyz=0 -8.2944E-05 0.08056 rpy=1.5708 0 0, axis 1 0 0, limit lower=-0.0047 upper=1E-05 effort=20.00001 velocity=2.00001

File: src/kuka_multiple_arms/robot_description/kuka_multiple_arms.xacro (robot description, xacro)
@@ -6,4 +6,5 @@
     <xacro:arg name="arm_id_3" default="kr3_disp_" />
     <xacro:arg name="arm_id_4" default="kr3_pip_" />
+    <xacro:arg name="arm_id_5" default="kr4_pp3_" />
     <!-- add gripper names prefixes -->
     <xacro:arg name="hand_id_1" default="schunk_" />
@@ -11,7 +12,9 @@
     <xacro:arg name="hand_id_3" default="kr3_disp_" />
     <xacro:arg name="hand_id_4" default="kr3_pip_" />
+    <xacro:arg name="hand_id_5" default="kr4_pp3_" />
     <!-- load arm/hand models and utils (which adds the robot inertia tags to be Gazebo-simulation ready) -->
     <!-- <xacro:include filename="$(find kuka_kr3_support)/urdf/kr3r540_macro_v2.xacro"/> -->
     <xacro:include filename="$(find kuka_kr3_support)/urdf/kr3r540_macro_v2.xacro"/>
+    <xacro:include filename="$(find kuka_kr4_support)/urdf/kr4r600_macro_v2.xacro"/>
     <xacro:include filename="$(find schunk_25nnb)/urdf/schunk_25nnb_macro.xacro"/>
     <link name="world"/>
@@ -56,4 +59,7 @@
     <xacro:kuka_kr3r540 prefix="$(arg arm_id_4)" connected_to="base"  xyz="1.9 0.5 1"  rpy="0 0 ${-pi}"/>
     <!-- <xacro:kuka_gripper arm_id="$(arg arm_id_2)" rpy="0 0 ${-pi/4}" connected_to="$(arg arm_id_2)_flange" /> -->
+    <!-- ROBOT 5 with gripper -->
+    <xacro:kuka_kr4r600 prefix="$(arg arm_id_5)" connected_to="base"  xyz="1.9 -1.5 1"  rpy="0 0 ${-pi}"/>
+    <xacro:schunk_25nnb prefix="$(arg arm_id_5)$(arg hand_id_5)"  rpy="0 0 ${-pi/2}" connected_to="$(arg arm_id_5)tool0" />
     <!-- <xacro:franka_arm arm_id="$(arg arm_id_2)" connected_to="base" xyz="0 0.5 1" gazebo="true" safety_distance="0.03" joint_limits="${xacro.load_yaml('$(find franka_description)/robots/panda/joint_limits.yaml')}"/>
     <xacro:franka_hand arm_id="$(arg arm_id_2)" rpy="0 0 ${-pi/4}" connected_to="$(arg arm_id_2)_link8" gazebo="true" safety_distance="0.03" /> -->

Commit message: Full xacro+urdf

File: src/kuka_multiple_arms/robot_description/kuka_multiple_arms.urdf (robot description, URDF)
Before this commit: robot kuka_multiple_arms, 57 links, 56 joints
Links:
- link base: geometry collision mesh filename=package://kuka_kr3_support/meshes/kr3r540/visual/TableNoDet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 scale=0.001 0.001 0.001; visual mesh filename=package://kuka_kr3_support/meshes/kr3r540/visual/TableNoDet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 scale=0.001 0.001 0.001
Joints:
- joint kr3_1__joint_base: origin xyz=0 -0.5 1 rpy=0 0 0 -> xyz=0.171 -1.16645 0 rpy=0 0 1.5707963267948966
- joint kr3_2__joint_base: origin xyz=0 0.5 1 rpy=0 0 0 -> xyz=0.729 -1.16645 0 rpy=0 0 1.5707963267948966
- joint kr3_3__joint_base: origin xyz=1.9 -0.5 1 rpy=0 0 -3.141592653589793 -> xyz=0.171 -0.20714 0 rpy=0 0 -1.5707963267948966
- joint kr3_4__joint_base: origin xyz=1.9 0.5 1 rpy=0 0 -3.141592653589793 -> xyz=0.729 -0.20714 0 rpy=0 0 -1.5707963267948966
- joint kr4_5__joint_base: origin xyz=1.9 -1.5 1 rpy=0 0 -3.141592653589793 -> xyz=1.37418 -0.20714 0 rpy=0 0 -1.5707963267948966

File: src/kuka_multiple_arms/robot_description/kuka_multiple_arms.xacro (robot description, xacro)
@@ -22,18 +22,26 @@
     <link name="base">
         <visual>
-            <origin xyz="0 0 0.5" rpy="0 0 0" />
-            <geometry>
-                <box size="1 2 1" />
-            </geometry>
-            <material name="White">
-                <color rgba="1.0 1.0 1.0 1.0" />
-            </material>
-        </visual>
-        <collision>
-            <origin xyz="0 0 0.5" rpy="0 0 0" />
-            <geometry>
-                <box size="1 2 1" />
-            </geometry>
-        </collision>
+        <origin
+          xyz="0 0 0"
+          rpy="0 0 0"/>
+        <geometry>
+          <mesh scale="0.001 0.001 0.001"
+            filename="package://kuka_kr3_support/meshes/kr3r540/visual/TableNoDetail.stl"/>
+        </geometry>
+        <material
+          name="">
+          <color
+            rgba="1 1 1 1" />
+        </material>
+      </visual>
+      <collision>
+        <origin
+          xyz="0 0 0"
+          rpy="0 0 0"/>
+        <geometry>
+          <mesh scale="0.001 0.001 0.001"
+            filename="package://kuka_kr3_support/meshes/kr3r540/visual/TableNoDetail.stl"/>
+        </geometry>
+      </collision>
         <inertial>
             <origin xyz="0.0 0.0 0.0" rpy="0.0 0.0 0.0"/>
@@ -48,17 +56,17 @@
     </joint>
     <!-- ROBOT 1 with gripper -->
-    <xacro:kuka_kr3r540 prefix="$(arg arm_id_1)" connected_to="base"  xyz="0 -0.5 1"  rpy="0 0 0"/>
+    <xacro:kuka_kr3r540 prefix="$(arg arm_id_1)" connected_to="base"  xyz="0.171 -1.16645 0"  rpy="0 0 ${pi/2}"/>
     <xacro:schunk_25nnb prefix="$(arg arm_id_1)$(arg hand_id_1)"  rpy="0 0 ${-pi/2}" connected_to="$(arg arm_id_1)tool0" />
     <!-- ROBOT 2 with gripper -->
-    <xacro:kuka_kr3r540 prefix="$(arg arm_id_2)" connected_to="base"  xyz="0 0.5 1" rpy="0 0 0" />
+    <xacro:kuka_kr3r540 prefix="$(arg arm_id_2)" connected_to="base"  xyz="0.729 -1.16645 0" rpy="0 0 ${pi/2}" />
     <xacro:schunk_25nnb prefix="$(arg arm_id_2)$(arg hand_id_2)"  rpy="0 0 ${-pi/2}" connected_to="$(arg arm_id_2)tool0" />
     <!-- ROBOT 3 with gripper -->
-    <xacro:kuka_kr3r540 prefix="$(arg arm_id_3)" connected_to="base"  xyz="1.9 -0.5 1"  rpy="0 0 ${-pi}"/>
+    <xacro:kuka_kr3r540 prefix="$(arg arm_id_3)" connected_to="base"  xyz="0.171 -0.20714 0"  rpy="0 0 ${-pi/2}"/>
     <xacro:pipette prefix="$(arg arm_id_3)$(arg hand_id_3)"  rpy="0 ${pi} ${-pi/2}" connected_to="$(arg arm_id_3)tool0" />
     <!-- ROBOT 4 with gripper -->
-    <xacro:kuka_kr3r540 prefix="$(arg arm_id_4)" connected_to="base"  xyz="1.9 0.5 1"  rpy="0 0 ${-pi}"/>
+    <xacro:kuka_kr3r540 prefix="$(arg arm_id_4)" connected_to="base"  xyz="0.729 -0.20714 0"  rpy="0 0 ${-pi/2}"/>
     <xacro:dispenser prefix="$(arg arm_id_4)$(arg hand_id_4)"  rpy="0 ${pi} ${-pi/2}" connected_to="$(arg arm_id_4)tool0" />
     <!-- ROBOT 5 with gripper -->
-    <xacro:kuka_kr4r600 prefix="$(arg arm_id_5)" connected_to="base"  xyz="1.9 -1.5 1"  rpy="0 0 ${-pi}"/>
+    <xacro:kuka_kr4r600 prefix="$(arg arm_id_5)" connected_to="base"  xyz="1.37418 -0.20714 0"  rpy="0 0 ${-pi/2}"/>
     <xacro:schunk_25nnb prefix="$(arg arm_id_5)$(arg hand_id_5)"  rpy="0 0 ${-pi/2}" connected_to="$(arg arm_id_5)tool0" />
 </robot>

Commit message: backup schunk 25nnb

File: src/kuka_multiple_arms/robot_description/kuka_multiple_arms.urdf (robot description, URDF)
Before this commit: robot kuka_multiple_arms, 57 links, 56 joints
Joints:
- joint kr3_1_schunk_base_joint: origin xyz=0 0 0 rpy=0 0 -1.5707963267948966 -> xyz=0 0 0 rpy=0 -1.5707963267948966 0
- joint kr3_2_schunk_base_joint: origin xyz=0 0 0 rpy=0 0 -1.5707963267948966 -> xyz=0 0 0 rpy=0 -1.5707963267948966 0
- joint kr4_5_schunk_base_joint: origin xyz=0 0 0 rpy=0 0 -1.5707963267948966 -> xyz=0 0 0 rpy=0 -1.5707963267948966 0
