Commit message: correct gripper orientation

File: src/kuka_multiple_arms/robot_description/kuka_multiple_arms.urdf (robot description, URDF)
Before this commit: robot kuka_multiple_arms, 57 links, 56 joints
Joints:
- joint kr3_1_schunk_base_joint: origin xyz=0 0 0 rpy=0 -1.5707963267948966 0 -> xyz=0 0 0 rpy=0 0 0
- joint kr3_2_schunk_base_joint: origin xyz=0 0 0 rpy=0 -1.5707963267948966 0 -> xyz=0 0 0 rpy=0 0 0
- joint kr4_5_schunk_base_joint: origin xyz=0 0 0 rpy=0 -1.5707963267948966 0 -> xyz=0 0 0 rpy=0 0 0

File: src/kuka_multiple_arms/robot_description/kuka_multiple_arms.xacro (robot description, xacro)
@@ -57,8 +57,8 @@
     <!-- ROBOT 1 with gripper -->
     <xacro:kuka_kr3r540 prefix="$(arg arm_id_1)" connected_to="base"  xyz="0.171 -1.16645 0"  rpy="0 0 ${pi/2}"/>
-    <xacro:schunk_25nnb prefix="$(arg arm_id_1)$(arg hand_id_1)"  rpy="0 ${-pi/2} 0" connected_to="$(arg arm_id_1)tool0" />
+    <xacro:schunk_25nnb prefix="$(arg arm_id_1)$(arg hand_id_1)"  rpy="0 0 0" connected_to="$(arg arm_id_1)tool0" />
     <!-- ROBOT 2 with gripper -->
     <xacro:kuka_kr3r540 prefix="$(arg arm_id_2)" connected_to="base"  xyz="0.729 -1.16645 0" rpy="0 0 ${pi/2}" />
-    <xacro:schunk_25nnb prefix="$(arg arm_id_2)$(arg hand_id_2)"  rpy="0 ${-pi/2} 0" connected_to="$(arg arm_id_2)tool0" />
+    <xacro:schunk_25nnb prefix="$(arg arm_id_2)$(arg hand_id_2)"  rpy="0 0 0" connected_to="$(arg arm_id_2)tool0" />
     <!-- ROBOT 3 with gripper -->
     <xacro:kuka_kr3r540 prefix="$(arg arm_id_3)" connected_to="base"  xyz="0.171 -0.20714 0"  rpy="0 0 ${-pi/2}"/>
@@ -69,4 +69,4 @@
     <!-- ROBOT 5 with gripper -->
     <xacro:kuka_kr4r600 prefix="$(arg arm_id_5)" connected_to="base"  xyz="1.37418 -0.20714 0"  rpy="0 0 ${-pi/2}"/>
-    <xacro:schunk_25nnb prefix="$(arg arm_id_5)$(arg hand_id_5)"  rpy="0 ${-pi/2} 0" connected_to="$(arg arm_id_5)tool0" />
+    <xacro:schunk_25nnb prefix="$(arg arm_id_5)$(arg hand_id_5)"  rpy="0 0 0" connected_to="$(arg arm_id_5)tool0" />
 </robot>

Commit message: new start joint positions

File: src/kuka_multiple_arms/robot_description/kuka_multiple_arms.urdf (robot description, URDF)
Before this commit: robot kuka_multiple_arms, 57 links, 56 joints
Joints:
- joint kr3_1_joint_a2: origin xyz=0.020 0 0 rpy=0 -1 0 -> xyz=0.020 0 0 rpy=0 -1.2 0
- joint kr3_1_joint_a3: origin xyz=0.260 0 0 rpy=0 0 0 -> xyz=0.260 0 0 rpy=0 1.8 0
- joint kr3_1_joint_a5: origin xyz=0.260 0 0 rpy=0 0 0 -> xyz=0.260 0 0 rpy=0 1 0
- joint kr3_2_joint_a2: origin xyz=0.020 0 0 rpy=0 -1 0 -> xyz=0.020 0 0 rpy=0 -1.2 0
- joint kr3_2_joint_a3: origin xyz=0.260 0 0 rpy=0 0 0 -> xyz=0.260 0 0 rpy=0 1.8 0
- joint kr3_2_joint_a5: origin xyz=0.260 0 0 rpy=0 0 0 -> xyz=0.260 0 0 rpy=0 1 0
- joint kr3_3_joint_a2: origin xyz=0.020 0 0 rpy=0 -1 0 -> xyz=0.020 0 0 rpy=0 -1.2 0
- joint kr3_3_joint_a3: origin xyz=0.260 0 0 rpy=0 0 0 -> xyz=0.260 0 0 rpy=0 1.8 0
- joint kr3_3_joint_a5: origin xyz=0.260 0 0 rpy=0 0 0 -> xyz=0.260 0 0 rpy=0 -0.55 0
- joint kr3_4_joint_a2: origin xyz=0.020 0 0 rpy=0 -1 0 -> xyz=0.020 0 0 rpy=0 -1.2 0
- joint kr3_4_joint_a3: origin xyz=0.260 0 0 rpy=0 0 0 -> xyz=0.260 0 0 rpy=0 1.8 0
- joint kr3_4_joint_a5: origin xyz=0.260 0 0 rpy=0 0 0 -> xyz=0.260 0 0 rpy=0 -0.55 0
- joint kr4_5_joint_a2: origin xyz=0.020 0 0 rpy=0 -1 0 -> xyz=0.020 0 0 rpy=0 -1.2 0
- joint kr4_5_joint_a3: origin xyz=0.290 0 0 rpy=0 0 0 -> xyz=0.290 0 0 rpy=0 1.8 0
- joint kr4_5_joint_a5: origin xyz=0 0 0 rpy=0 0 0 -> xyz=0 0 0 rpy=0 1 0

Commit message: default start joint positions

File: src/kuka_multiple_arms/robot_description/kuka_multiple_arms.urdf (robot description, URDF)
Before this commit: robot kuka_multiple_arms, 57 links, 56 joints
Joints:
- joint kr3_1_joint_a2: origin xyz=0.020 0 0 rpy=0 -1.2 0 -> xyz=0.020 0 0 rpy=0 -1 0
- joint kr3_1_joint_a3: origin xyz=0.260 0 0 rpy=0 1.8 0 -> xyz=0.260 0 0 rpy=0 0 0
- joint kr3_1_joint_a5: origin xyz=0.260 0 0 rpy=0 1 0 -> xyz=0.260 0 0 rpy=0 0 0
- joint kr3_2_joint_a2: origin xyz=0.020 0 0 rpy=0 -1.2 0 -> xyz=0.020 0 0 rpy=0 -1 0
- joint kr3_2_joint_a3: origin xyz=0.260 0 0 rpy=0 1.8 0 -> xyz=0.260 0 0 rpy=0 0 0
- joint kr3_2_joint_a5: origin xyz=0.260 0 0 rpy=0 1 0 -> xyz=0.260 0 0 rpy=0 0 0
- joint kr3_3_joint_a2: origin xyz=0.020 0 0 rpy=0 -1.2 0 -> xyz=0.020 0 0 rpy=0 -1 0
- joint kr3_3_joint_a3: origin xyz=0.260 0 0 rpy=0 1.8 0 -> xyz=0.260 0 0 rpy=0 0 0
- joint kr3_3_joint_a5: origin xyz=0.260 0 0 rpy=0 -0.55 0 -> xyz=0.260 0 0 rpy=0 0 0
- joint kr3_4_joint_a2: origin xyz=0.020 0 0 rpy=0 -1.2 0 -> xyz=0.020 0 0 rpy=0 -1 0
- joint kr3_4_joint_a3: origin xyz=0.260 0 0 rpy=0 1.8 0 -> xyz=0.260 0 0 rpy=0 0 0
- joint kr3_4_joint_a5: origin xyz=0.260 0 0 rpy=0 -0.55 0 -> xyz=0.260 0 0 rpy=0 0 0
- joint kr4_5_joint_a2: origin xyz=0.020 0 0 rpy=0 -1.2 0 -> xyz=0.020 0 0 rpy=0 -1 0
- joint kr4_5_joint_a3: origin xyz=0.290 0 0 rpy=0 1.8 0 -> xyz=0.290 0 0 rpy=0 0 0
- joint kr4_5_joint_a5: origin xyz=0 0 0 rpy=0 1 0 -> xyz=0 0 0 rpy=0 0 0
